File: circuits/VCO.brd (EAGLE design)
At the start: 100 x 80 mm, 25 parts, among them Q1 16MHZ

Commit message: circuits changes
Parts:
- moved LFO4 15.2 mm to (59.7, 3.81)
- moved C1 15.2 mm to (29.2, 12.7)
- moved C4 15.2 mm to (34.3, 39.4)
- moved FTDI 15.2 mm to (2.54, 19.1)
- moved LFO1 15.2 mm to (31.8, 3.81)
- moved LFO2 15.2 mm to (40.6, 3.81)
- moved Q1 15.2 mm to (40.6, 12.7)
- moved C5 15.2 mm to (3.81, 30.5)
- moved VCIN 15.2 mm to (14.0, 41.9)
- moved PWR1 15.2 mm to (8.89, 12.7)
- moved R1 15.2 mm to (19.1, 11.4)
- moved STATUS 15.2 mm to (21.6, 3.81)
- moved C2 15.2 mm to (33.0, 12.7)
- moved C3 15.2 mm to (49.5, 12.7)
- moved FUTURE 15.2 mm to (54.6, 41.9)
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Other:
- board size 100 x 80 mm -> 84.8 x 45.7 mm
