File: modules/divider/circuits/divider.brd (EAGLE design)
At the start: 37.8 x 52.1 mm, 28 parts

Commit message: adding clock module
Parts:
- removed R41, R42, R43, R44, R45, R46, R47: 1k, SparkFun-Resistors:AXIAL-0.3
- removed WIDTH_SELECTION1: (no value), pinhead:2X07
- added JP1: (no value), pinhead:2X08
- moved R56 10.2 mm to (35.6, 40.6), turned to 270 degrees
- moved R40 7.73 mm to (38.1, 40.6), turned to 90 degrees
Connections:
- removed net N$62: R41.P$2, R47.P$1, R49.P$2, WIDTH_SELECTION1.13
- new net N$1: JP1.4, R49.P$2
- new net N$2: JP1.2, R48.P$2
- net GATE_OUT: now also JP1.1, JP1.11, JP1.13, JP1.15, JP1.3, JP1.5, JP1.7, JP1.9, R56.P$2; no longer R47.P$2, R48.P$2, R56.P$1
- net GNDA: now also R56.P$1; no longer R56.P$2, WIDTH_SELECTION1.10, WIDTH_SELECTION1.12, WIDTH_SELECTION1.14, WIDTH_SELECTION1.2, WIDTH_SELECTION1.4, WIDTH_SELECTION1.6, WIDTH_SELECTION1.8
- net N$63: now also JP1.6; no longer R41.P$1, R42.P$2, WIDTH_SELECTION1.11
- net N$65: now also JP1.10; no longer R43.P$1, R44.P$2, WIDTH_SELECTION1.7
- net N$66: now also JP1.12; no longer R44.P$1, R45.P$2, WIDTH_SELECTION1.5
- net N$67: now also JP1.14; no longer R45.P$1, R46.P$2, WIDTH_SELECTION1.3
- net N$68: now also JP1.16; no longer R46.P$1, WIDTH_SELECTION1.1
- net N$71: now also JP1.8; no longer R42.P$1, R43.P$2, WIDTH_SELECTION1.9
Routing:
- net N$68: track 48.4 -> 7.40 mm
- net GNDA: track 56.7 -> 16.6 mm
- net N$66: track 47.3 -> 7.40 mm
- net N$67: track 43.4 -> 7.40 mm
- net N$71: track 34.6 -> 7.40 mm
- net N$62: track 25.2 -> 0.00 mm
- net N$65: track 31.4 -> 7.40 mm
- net GATE_OUT: track 25.2 -> 40.9 mm
- net N$63: track 23.0 -> 7.40 mm
- net DIV8_CLK: track 33.1 -> 25.3 mm
- net N$1: track 0.00 -> 7.40 mm
- net N$2: track 0.00 -> 7.40 mm
Other:
- board size 37.8 x 52.1 mm -> 34 x 48.2 mm
- board text removed: "1/8"
- board text removed: "2/8"
- board text removed: "3/8"
- board text removed: "4/8"
- board text removed: "5/8"
- board text removed: "6/8"
- board text removed: "7/8"
