File: modules/sequencer/circuits/sequencer.brd (EAGLE design)
At the start: 68.2 x 80 mm, 56 parts, among them IC1 LM555N, IC2 LM324N

Commit message: midi2cv
Parts:
- removed 1K2, 1K6: 1k, adafruit:0207/12
- removed 1K5: 10k, adafruit:0207/12
- removed 2N3: (no value), transistor-neu-to92:TO92-EBC
- removed JP1: (no value), pinhead:2X03
- added IC3: 4056N, 40xx:DIL16
- added R24: 10k, adafruit:0207/12
- C2: value 220uf -> 100uf
Connections:
- removed net COUNTER_POWER: IC2.8, IC2.9
- removed net N$37: 1K5.2, 2N3.B
- removed net N$38: 1K5.1, JP1.4, V1.11
- removed net N$39: 1K2.2, 1K6.2, 2N3.C
- removed net N$40: 1K2.1, JP1.6
- removed net N$42: IC2.10, JP1.1, JP1.3, JP1.5
- new net VCC: IC3.16
- new net VEE: IC3.7
- net 5V: now also V1.1, V1.10, V1.7, V1.9; no longer 1K6.1, JP1.2
- net CLK_IN: now also R24.1
- net GND: now also IC3.4, IC3.8, R24.2; no longer 2N3.E
Changed lines of the file:
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@@
 <?xml version="1.0" encoding="utf-8"?>
 <!DOCTYPE eagle SYSTEM "eagle.dtd">
-<eagle version="9.5.2">
+<eagle version="9.6.2">
 <drawing>
 <settings>
@@
 <attribute name="VALUE" x="62.23" y="4.445" size="1.27" layer="27"/>
 </element>
-<element name="C2" library="rcl" library_urn="urn:adsk.eagle:library:334" package="E2,5-6E" package3d_urn="urn:adsk.eagle:package:23430/1" value="220uf" x="71.12" y="27.94" smashed="yes">
+<element name="C2" library="rcl" library_urn="urn:adsk.eagle:library:334" package="E2,5-6E" package3d_urn="urn:adsk.eagle:package:23430/1" value="100uf" x="71.12" y="27.94" smashed="yes">
 <attribute name="POPULARITY" value="1" x="71.12" y="27.94" size="1.778" layer="27" display="off"/>
 <attribute name="SPICEPREFIX" value="C" x="71.12" y="27.94" size="1.778" layer="27" display="off"/>
@@
 <attribute name="VALUE" x="11.938" y="-176.784" size="1.27" layer="27" ratio="10"/>
 </element>
-<element name="1K2" library="adafruit" library_urn="urn:adsk.eagle:library:420" package="0207/12" package3d_urn="urn:adsk.eagle:package:6240598/1" value="1k" x="7.62" y="-181.61" smashed="yes">
-<attribute name="NAME" x="4.445" y="-180.213" size="1.27" layer="25" ratio="10"/>
-<attribute name="VALUE" x="5.334" y="-182.2958" size="1.27" layer="27" ratio="10"/>
-</element>
 <element name="V1" library="74ttl-din" library_urn="urn:adsk.eagle:library:84" package="DIL16" package3d_urn="urn:adsk.eagle:package:922/2" value="74161N" x="12.7" y="-189.23" smashed="yes">
 <attribute name="NAME" x="2.159" y="-192.151" size="1.27" layer="25" ratio="10" rot="R90"/>
@@
 <attribute name="VALUE" x="5.207" y="-189.865" size="1.27" layer="27" ratio="10"/>
 </element>
-<element name="2N3" library="transistor-neu-to92" library_urn="urn:adsk.eagle:library:397" package="TO92-EBC" package3d_urn="urn:adsk.eagle:package:28763/2" value="" x="-6.35" y="-193.04" smashed="yes">
-<attribute name="NAME" x="-8.89" y="-191.262" size="1.27" layer="25" ratio="10"/>
-<attribute name="POPULARITY" value="0" x="-6.35" y="-193.04" size="1.778" layer="27" display="off"/>
-<attribute name="VALUE" x="-8.89" y="-197.612" size="1.27" layer="27" ratio="10"/>
-</element>
-<element name="1K6" library="adafruit" library_urn="urn:adsk.eagle:library:420" package="0207/12" package3d_urn="urn:adsk.eagle:package:6240598/1" value="1k" x="-1.27" y="-203.2" smashed="yes">
-<attribute name="NAME" x="-4.445" y="-201.803" size="1.27" layer="25" ratio="10"/>
-<attribute name="VALUE" x="-3.556" y="-203.8858" size="1.27" layer="27" ratio="10"/>
-</element>
-<element name="JP1" library="pinhead" library_urn="urn:adsk.eagle:library:325" package="2X03" package3d_urn="urn:adsk.eagle:package:22462/2" value="" x="-13.97" y="-199.39" smashed="yes">
-<attribute name="NAME" x="-17.78" y="-196.215" size="1.27" layer="25" ratio="10"/>
-<attribute name="POPULARITY" value="62" x="-13.97" y="-199.39" size="1.778" layer="27" display="off"/>
-<attribute name="VALUE" x="-17.78" y="-203.835" size="1.27" layer="27"/>
-</element>
-<element name="1K5" library="adafruit" library_urn="urn:adsk.eagle:library:420" package="0207/12" package3d_urn="urn:adsk.eagle:package:6240598/1" value="10k" x="-10.16" y="-208.28" smashed="yes">
-<attribute name="NAME" x="-13.335" y="-206.883" size="1.27" layer="25" ratio="10"/>
-<attribute name="VALUE" x="-12.446" y="-208.9658" size="1.27" layer="27" ratio="10"/>
+<element name="R24" library="adafruit" library_urn="urn:adsk.eagle:library:420" package="0207/12" package3d_urn="urn:adsk.eagle:package:6240598/1" value="10k" x="7.62" y="-198.12" smashed="yes">
+<attribute name="NAME" x="4.445" y="-196.723" size="1.27" layer="25" ratio="10"/>
+<attribute name="VALUE" x="5.334" y="-198.8058" size="1.27" layer="27" ratio="10"/>
+</element>
+<element name="IC3" library="40xx" library_urn="urn:adsk.eagle:library:80" package="DIL16" package3d_urn="urn:adsk.eagle:package:922/2" value="4056N" x="12.7" y="-205.74" smashed="yes">
+<attribute name="NAME" x="2.159" y="-208.661" size="1.27" layer="25" ratio="10" rot="R90"/>
+<attribute name="POPULARITY" value="0" x="12.7" y="-205.74" size="1.778" layer="27" display="off"/>
+<attribute name="VALUE" x="5.207" y="-206.375" size="1.27" layer="27" ratio="10"/>
 </element>
 </elements>
@@
 <wire x1="60.96" y1="12.7" x2="60.96" y2="10.16" width="0.1524" layer="1"/>
 <contactref element="R23" pad="1"/>
-<contactref element="2N3" pad="E"/>
-<wire x1="8.89" y1="-156.21" x2="-8.89" y2="-194.31" width="0" layer="19" extent="1-1"/>
+<contactref element="R24" pad="2"/>
+<contactref element="IC3" pad="8"/>
+<contactref element="IC3" pad="4"/>
+<wire x1="21.59" y1="-209.55" x2="11.43" y2="-209.55" width="0" layer="19" extent="1-1"/>
+<wire x1="13.97" y1="-198.12" x2="11.43" y2="-209.55" width="0" layer="19" extent="1-1"/>
+<wire x1="8.89" y1="-156.21" x2="13.97" y2="-198.12" width="0" layer="19" extent="1-1"/>
 <wire x1="11.43" y1="-135.89" x2="8.89" y2="-156.21" width="0" layer="19" extent="1-1"/>
 <wire x1="11.43" y1="-130.81" x2="11.43" y2="-135.89" width="0" layer="19" extent="1-1"/>
@@
 <contactref element="C2" pad="+"/>
 <contactref element="D1" pad="C"/>
-<contactref element="1K6" pad="1"/>
-<contactref element="JP1" pad="2"/>
-<wire x1="-7.62" y1="-203.2" x2="-16.51" y2="-198.12" width="0" layer="19" extent="1-1"/>
-<wire x1="8.89" y1="-173.99" x2="-7.62" y2="-203.2" width="0" layer="19" extent="1-1"/>
+<contactref element="V1" pad="9"/>
+<contactref element="V1" pad="10"/>
+<contactref element="V1" pad="7"/>
+<contactref element="V1" pad="1"/>
+<wire x1="19.05" y1="-193.04" x2="3.81" y2="-193.04" width="0" layer="19" extent="1-1"/>
+<wire x1="19.05" y1="-185.42" x2="19.05" y2="-193.04" width="0" layer="19" extent="1-1"/>
+<wire x1="21.59" y1="-185.42" x2="19.05" y2="-185.42" width="0" layer="19" extent="1-1"/>
+<wire x1="8.89" y1="-173.99" x2="19.05" y2="-185.42" width="0" layer="19" extent="1-1"/>
 <wire x1="19.05" y1="-130.81" x2="8.89" y2="-173.99" width="0" layer="19" extent="1-1"/>
 <wire x1="11.43" y1="-123.19" x2="19.05" y2="-130.81" width="0" layer="19" extent="1-1"/>
@@
 <contactref element="2N2" pad="B"/>
 <contactref element="V1" pad="2"/>
+<contactref element="R24" pad="1"/>
+<wire x1="6.35" y1="-193.04" x2="1.27" y2="-198.12" width="0" layer="19" extent="1-1"/>
 <wire x1="19.05" y1="3.81" x2="6.35" y2="-193.04" width="0" layer="19" extent="1-1"/>
 <wire x1="10.16" y1="7.62" x2="19.05" y2="3.81" width="0" layer="19" extent="1-1"/>
@@
 <contactref element="V1" pad="8"/>
 </signal>
-<signal name="N$38">
-<contactref element="V1" pad="11"/>
-<contactref element="JP1" pad="4"/>
-<contactref element="1K5" pad="1"/>
-<wire x1="-13.97" y1="-198.12" x2="-16.51" y2="-208.28" width="0" layer="19" extent="1-1"/>
-<wire x1="16.51" y1="-185.42" x2="-13.97" y2="-198.12" width="0" layer="19" extent="1-1"/>
-</signal>
-<signal name="N$39">
-<contactref element="1K6" pad="2"/>
-<contactref element="2N3" pad="C"/>
-<contactref element="1K2" pad="2"/>
-<wire x1="-3.81" y1="-194.31" x2="5.08" y2="-203.2" width="0" layer="19" extent="1-1"/>
-<wire x1="13.97" y1="-181.61" x2="-3.81" y2="-194.31" width="0" layer="19" extent="1-1"/>
-</signal>
-<signal name="N$40">
-<contactref element="1K2" pad="1"/>
-<contactref element="JP1" pad="6"/>
-<wire x1="1.27" y1="-181.61" x2="-11.43" y2="-198.12" width="0" layer="19" extent="1-1"/>
-</signal>
-<signal name="N$42">
-<contactref element="JP1" pad="5"/>
-<contactref element="JP1" pad="3"/>
-<contactref element="JP1" pad="1"/>
-<contactref element="IC2" pad="10"/>
-<wire x1="-13.97" y1="-200.66" x2="-16.51" y2="-200.66" width="0" layer="19" extent="1-1"/>
-<wire x1="-11.43" y1="-200.66" x2="-13.97" y2="-200.66" width="0" layer="19" extent="1-1"/>
-<wire x1="22.86" y1="13.97" x2="-11.43" y2="-200.66" width="0" layer="19" extent="1-1"/>
-</signal>
-<signal name="COUNTER_POWER">
-<contactref element="IC2" pad="8"/>
-<contactref element="IC2" pad="9"/>
-<wire x1="17.78" y1="13.97" x2="20.32" y2="13.97" width="0" layer="19" extent="1-1"/>
-</signal>
-<signal name="N$37">
-<contactref element="2N3" pad="B"/>
-<contactref element="1K5" pad="2"/>
-<wire x1="-6.35" y1="-194.31" x2="-3.81" y2="-208.28" width="0" layer="19" extent="1-1"/>
-</signal>
 <signal name="Q1">
 <contactref element="V1" pad="14"/>
@@
 <contactref element="V1" pad="12"/>
 </signal>
+<signal name="VEE">
+<contactref element="IC3" pad="7"/>
+</signal>
+<signal name="VCC">
+<contactref element="IC3" pad="16"/>
+</signal>
 </signals>

Commit message: sequencer board
Parts:
- removed LED1, LED2, LED3, LED4, LED5, LED6, LED7, LED8: (no value), adafruit:LED5MM
- removed R19: 330, adafruit:0207/12
- added D2: 157119S12801, Wurth_7 Segments Display_WL-T7DS:WL-T7DS_0.39INCH
- moved IC3 267.5 mm to (45.7, 59.7), turned to 180 degrees
- moved V1 262.4 mm to (45.7, 71.1), turned to 180 degrees
- moved R24 207.2 mm to (16.5, 8.89), turned to 180 degrees
- moved R23 195.8 mm to (54.6, 35.6), turned to 270 degrees
- moved D1 192.2 mm to (39.4, 16.5), turned to 90 degrees
- moved C4 188.6 mm to (36.8, 20.3), turned to 270 degrees
- moved LED9 177.7 mm to (53.3, 24.1)
- moved 1K1 172.7 mm to (16.5, 11.4), turned to 180 degrees
- moved R21 149.7 mm to (48.3, 2.54)
- moved IC1 146.3 mm to (49.5, 15.2), turned to 270 degrees
- moved C1 140.7 mm to (26.7, 3.81), turned to 180 degrees
- moved RESET_BUTTON 58.9 mm to (15.2, 54.6), turned to 180 degrees
- moved 1K4 47.8 mm to (30.5, 8.89)
- moved 1K3 47.8 mm to (33.0, 8.89), turned to 270 degrees
- moved 2N2 41.3 mm to (27.9, 12.7), turned to 270 degrees
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Connections:
- removed net +UB: V1.16
- removed net -UB: V1.8
- removed net VCC: IC3.16
- removed net VEE: IC3.7
- new net N$37: IC3.9, R1.1
- new net N$38: IC3.10, R13.1
- new net N$39: IC3.11, R14.1
- new net N$40: IC3.12, R15.1
- new net N$41: IC3.13, R16.1
- new net N$42: IC3.14, R18.1
- net 5V: now also D2.3, D2.8, IC3.1, IC3.16, IC3.6, V1.16
- net GND: now also IC3.7, V1.8; no longer LED1.K, LED2.K, LED3.K, LED4.K, LED5.K, LED6.K, LED7.K, LED8.K
- net N$22: now also IC3.15, R17.1; no longer LED3.A, R14.1
- net N$23: now also D2.1, R18.2; no longer LED4.A, R15.1
- net N$24: now also D2.2, R17.2; no longer LED5.A, R16.1
- net N$25: now also D2.4, R16.2; no longer LED6.A, R17.1
- net N$26: now also D2.5, R15.2; no longer LED7.A, R18.1
- net N$27: now also D2.7, R14.2; no longer LED8.A, R19.1
- net N$28: now also D2.9, R13.2; no longer LED2.A, R13.1
- net N$29: now also D2.10, R1.2; no longer LED1.A, R1.1
- net Q1: now also IC3.5
- net Q2: now also IC3.3
- net Q3: now also IC3.2
Routing:
- net 5V: track 66.7 -> 276.6 mm
- net CV_OUT: track 56.9 -> 19.1 mm
- net N$36: track 0.00 -> 36.7 mm
- net CLK_IN: track 183.1 -> 149.4 mm
- net GND: track 225.5 -> 257.1 mm
- net N$10: track 59.2 -> 27.8 mm
- net N$34: track 0.00 -> 29.6 mm
- net N$9: track 44.8 -> 21.7 mm
- net N$28: track 8.45 -> 29.6 mm
- net Q3: track 0.00 -> 20.8 mm
- net N$7: track 50.1 -> 29.3 mm, vias 1 -> 0
- net N$35: track 0.00 -> 19.6 mm
- net N$5: track 51.6 -> 32.9 mm
- net N$8: track 38.7 -> 21.7 mm
- net N$32: track 0.00 -> 14.0 mm
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Other:
- board size 68.2 x 80 mm -> 49.2 x 78.7 mm
