File: modules/sequencer/circuits/sequencer.brd (EAGLE design)
At the start: 49.2 x 78.7 mm, 45 parts, among them IC1 LM555N, IC2 LM324N, IC3 4056N

Commit message: uni2bi
Parts:
- removed C2: 100uf, rcl:E2,5-6E
- added C3: 100uf, rcl:E2,5-6E
Connections:
- net 5V: now also GATE_POT.1; no longer C2.+
- net GND: now also C3.-; no longer GATE_POT.1
- net N$35: now also C3.+; no longer C2.-
Routing:
- net GND: track 257.1 -> 262.4 mm
- net 5V: track 276.6 -> 278.4 mm
- net N$33: track 14.0 -> 12.5 mm
- net N$35: track 19.6 -> 20.6 mm
- net CV_OUT: track 19.1 -> 19.9 mm
Other:
- board text added: "+12"
- board text added: "+5"
- board text added: "-12"
- board text added: "10k"
- board text added: "CLK"
- board text added: "DUMAIS SEQUENCER"
- board text added: "GND"

Commit message: Sequencer fixes
Parts:
- added R19: 1K, adafruit:0207/12
Connections:
- new net N$43: 2N2.B, R19.1
- net CLK_IN: now also R19.2; no longer 2N2.B
Routing:
- net CLK_IN: track 149.4 -> 144.4 mm
Changed lines of the file:
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@@
 <attribute name="VALUE" x="45.593" y="8.89" size="1.27" layer="25" ratio="10" rot="R180"/>
+</element>
+<element name="R19" library="adafruit" library_urn="urn:adsk.eagle:library:420" package="0207/12" package3d_urn="urn:adsk.eagle:package:6240598/1" value="1K" x="15.24" y="-119.38" smashed="yes">
+<attribute name="NAME" x="12.065" y="-117.983" size="1.27" layer="25" ratio="10"/>
+<attribute name="VALUE" x="12.954" y="-120.0658" size="1.27" layer="27" ratio="10"/>
 </element>
 </elements>
@@
 <contactref element="INPUTS1" pad="5"/>
 <contactref element="CD4017" pad="14"/>
-<contactref element="2N2" pad="B"/>
 <contactref element="V1" pad="2"/>
 <contactref element="R24" pad="1"/>
@@
 <wire x1="15.11374375" y1="72.6948" x2="16.8148" y2="72.6948" width="0.1524" layer="16"/>
 <wire x1="11.2522" y1="72.39" x2="14.80894375" y2="72.39" width="0.1524" layer="16"/>
-<wire x1="26.67" y1="12.7" x2="21.59" y2="12.7" width="0.1524" layer="1"/>
 <wire x1="21.59" y1="12.7" x2="20.32" y2="11.43" width="0.1524" layer="1"/>
 <wire x1="20.32" y1="11.43" x2="20.32" y2="3.81" width="0.1524" layer="1"/>
 <wire x1="22.86" y1="8.89" x2="20.32" y2="8.89" width="0.1524" layer="1"/>
 <wire x1="20.32" y1="8.89" x2="20.32" y2="3.81" width="0.1524" layer="1"/>
+<contactref element="R19" pad="2"/>
+<wire x1="20.32" y1="3.81" x2="21.59" y2="-119.38" width="0" layer="19" extent="1-1"/>
 </signal>
 <signal name="N$3">
@@
 <wire x1="49.53" y1="53.34" x2="49.53" y2="55.88" width="0.1524" layer="1"/>
 </signal>
+<signal name="N$43">
+<contactref element="2N2" pad="B"/>
+<contactref element="R19" pad="1"/>
+<wire x1="26.67" y1="12.7" x2="8.89" y2="-119.38" width="0" layer="19" extent="1-1"/>
+</signal>
 </signals>
