File: modules/sequencer/circuits/sequencer.sch (EAGLE design)
At the start: 45 parts, among them IC1 LM555N, IC2 LM324N, IC3 4056N

Commit message: uni2bi
Parts:
- removed C2: 100uf, rcl:CPOL-USE2,5-6E
- added C3: 100uf, rcl:CPOL-USE2,5-6E
Connections:
- net 5V: now also GATE_POT.1; no longer C2.+
- net GND: now also C3.-; no longer GATE_POT.1
- net N$35: now also C3.+; no longer C2.-
Changed lines of the file:
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@@
 <?xml version="1.0" encoding="utf-8"?>
 <!DOCTYPE eagle SYSTEM "eagle.dtd">
-<eagle version="9.5.2">
+<eagle version="9.6.2">
 <drawing>
 <settings>
@@
 <part name="R20" library="adafruit" library_urn="urn:adsk.eagle:library:420" deviceset="R-US_" device="0207/12" package3d_urn="urn:adsk.eagle:package:6240598/1" value="10k"/>
 <part name="1K3" library="adafruit" library_urn="urn:adsk.eagle:library:420" deviceset="R-US_" device="0207/12" package3d_urn="urn:adsk.eagle:package:6240598/1" value="1k"/>
-<part name="SUPPLY1" library="SparkFun-PowerSymbols" library_urn="urn:adsk.eagle:library:530" deviceset="5V" device=""/>
 <part name="GATE_POT" library="pinhead" library_urn="urn:adsk.eagle:library:325" deviceset="PINHD-1X2" device="" package3d_urn="urn:adsk.eagle:package:22435/2"/>
-<part name="C2" library="rcl" library_urn="urn:adsk.eagle:library:334" deviceset="CPOL-US" device="E2,5-6E" package3d_urn="urn:adsk.eagle:package:23430/1" value="100uf"/>
 <part name="1K4" library="adafruit" library_urn="urn:adsk.eagle:library:420" deviceset="R-US_" device="0207/12" package3d_urn="urn:adsk.eagle:package:6240598/1" value="10k"/>
 <part name="GND11" library="supply1" library_urn="urn:adsk.eagle:library:371" deviceset="GND" device=""/>
@@
 <part name="SUPPLY7" library="SparkFun-PowerSymbols" library_urn="urn:adsk.eagle:library:530" deviceset="5V" device=""/>
 <part name="C1" library="rcl" library_urn="urn:adsk.eagle:library:334" deviceset="C-EU" device="025-024X044" package3d_urn="urn:adsk.eagle:package:23630/1" value="0.01uf"/>
-<part name="GND5" library="supply1" library_urn="urn:adsk.eagle:library:371" deviceset="GND" device=""/>
 <part name="R21" library="adafruit" library_urn="urn:adsk.eagle:library:420" deviceset="R-US_" device="0207/12" package3d_urn="urn:adsk.eagle:package:6240598/1" value="100"/>
 <part name="LED9" library="adafruit" library_urn="urn:adsk.eagle:library:420" deviceset="LED" device="5MM" package3d_urn="urn:adsk.eagle:package:6240538/1"/>
@@
 <part name="GND10" library="supply1" library_urn="urn:adsk.eagle:library:371" deviceset="GND" device=""/>
 <part name="SUPPLY15" library="SparkFun-PowerSymbols" library_urn="urn:adsk.eagle:library:530" deviceset="5V" device=""/>
+<part name="GND14" library="supply1" library_urn="urn:adsk.eagle:library:371" deviceset="GND" device=""/>
+<part name="SUPPLY13" library="SparkFun-PowerSymbols" library_urn="urn:adsk.eagle:library:530" deviceset="5V" device=""/>
+<part name="C3" library="rcl" library_urn="urn:adsk.eagle:library:334" deviceset="CPOL-US" device="E2,5-6E" package3d_urn="urn:adsk.eagle:package:23430/1" value="100uf"/>
 </parts>
 <sheets>
@@
 <wire x1="170.18" y1="15.24" x2="53.34" y2="15.24" width="0.1524" layer="152" style="shortdash"/>
 <wire x1="53.34" y1="15.24" x2="-58.42" y2="15.24" width="0.1524" layer="152" style="shortdash"/>
-<wire x1="170.18" y1="15.24" x2="172.72" y2="-96.52" width="0.1524" layer="152" style="shortdash"/>
+<wire x1="170.18" y1="15.24" x2="170.18" y2="-96.52" width="0.1524" layer="152" style="shortdash"/>
 <wire x1="170.18" y1="15.24" x2="170.18" y2="116.84" width="0.1524" layer="152" style="shortdash"/>
 <wire x1="170.18" y1="15.24" x2="340.36" y2="15.24" width="0.1524" layer="152" style="shortdash"/>
@@
 <attribute name="VALUE" x="209.55" y="-62.738" size="1.778" layer="96" rot="R180"/>
 </instance>
-<instance part="SUPPLY1" gate="G$1" x="312.42" y="-55.88" smashed="yes">
-<attribute name="VALUE" x="312.42" y="-50.546" size="1.778" layer="96" rot="R90" align="bottom-center"/>
-</instance>
 <instance part="GATE_POT" gate="G$1" x="309.88" y="-88.9" smashed="yes" rot="R180">
 <attribute name="NAME" x="318.77" y="-84.455" size="1.778" layer="95" rot="R270"/>
 <attribute name="VALUE" x="316.23" y="-83.82" size="1.778" layer="96" rot="R180"/>
-</instance>
-<instance part="C2" gate="G$1" x="312.42" y="-60.96" smashed="yes">
-<attribute name="VALUE" x="318.516" y="-65.151" size="1.778" layer="96" rot="R90"/>
 </instance>
 <instance part="1K4" gate="G$1" x="198.12" y="-50.8" smashed="yes" rot="R90">
@@
 <attribute name="VALUE" x="245.364" y="-75.819" size="1.778" layer="96"/>
 </instance>
-<instance part="GND5" gate="1" x="312.42" y="-101.6" smashed="yes"/>
 <instance part="R21" gate="G$1" x="312.42" y="-78.74" smashed="yes" rot="R90">
 <attribute name="VALUE" x="310.642" y="-80.01" size="1.778" layer="96" rot="R90"/>
@@
 <attribute name="VALUE" x="172.466" y="38.1" size="1.778" layer="96" rot="R180" align="bottom-center"/>
 </instance>
+<instance part="GND14" gate="1" x="327.66" y="-63.5" smashed="yes"/>
+<instance part="SUPPLY13" gate="G$1" x="312.42" y="-99.06" smashed="yes" rot="R180">
+<attribute name="VALUE" x="312.42" y="-104.394" size="1.778" layer="96" rot="R270" align="bottom-center"/>
+</instance>
+<instance part="C3" gate="G$1" x="312.42" y="-63.5" smashed="yes" rot="R180">
+<attribute name="VALUE" x="306.324" y="-59.309" size="1.778" layer="96" rot="R270"/>
+</instance>
 </instances>
 <busses>
@@
 </segment>
 <segment>
-<pinref part="GATE_POT" gate="G$1" pin="1"/>
-<wire x1="312.42" y1="-99.06" x2="312.42" y2="-91.44" width="0.1524" layer="91"/>
-<pinref part="GND5" gate="1" pin="GND"/>
-</segment>
-<segment>
 <pinref part="R23" gate="G$1" pin="1"/>
 <pinref part="GND6" gate="1" pin="GND"/>
@@
 <junction x="200.66" y="33.02"/>
 </segment>
+<segment>
+<wire x1="312.42" y1="-58.42" x2="312.42" y2="-55.88" width="0.1524" layer="91"/>
+<pinref part="GND14" gate="1" pin="GND"/>
+<wire x1="312.42" y1="-55.88" x2="327.66" y2="-55.88" width="0.1524" layer="91"/>
+<wire x1="327.66" y1="-55.88" x2="327.66" y2="-60.96" width="0.1524" layer="91"/>
+<pinref part="C3" gate="G$1" pin="-"/>
+</segment>
 </net>
 <net name="12V" class="0">
@@
 </net>
 <net name="5V" class="0">
-<segment>
-<pinref part="SUPPLY1" gate="G$1" pin="5V"/>
-<wire x1="312.42" y1="-58.42" x2="312.42" y2="-55.88" width="0.1524" layer="91"/>
-<pinref part="C2" gate="G$1" pin="+"/>
-</segment>
 <segment>
 <pinref part="CD4017" gate="G2" pin="P$V+"/>
@@
 <pinref part="IC3" gate="P" pin="VCC"/>
 <wire x1="177.8" y1="38.1" x2="182.88" y2="38.1" width="0.1524" layer="91"/>
+</segment>
+<segment>
+<pinref part="GATE_POT" gate="G$1" pin="1"/>
+<wire x1="312.42" y1="-99.06" x2="312.42" y2="-91.44" width="0.1524" layer="91"/>
+<pinref part="SUPPLY13" gate="G$1" pin="5V"/>
 </segment>
 </net>
@@
 <wire x1="312.42" y1="-68.58" x2="312.42" y2="-73.66" width="0.1524" layer="91"/>
 <pinref part="R21" gate="G$1" pin="2"/>
-<pinref part="C2" gate="G$1" pin="-"/>
 <wire x1="312.42" y1="-66.04" x2="312.42" y2="-68.58" width="0.1524" layer="91"/>
 <junction x="312.42" y="-68.58"/>
-</segment>
-</net>
+<pinref part="C3" gate="G$1" pin="+"/>
+</segment>
+</net>

Commit message: Sequencer fixes
Parts:
- added R19: 1K, adafruit:R-US_0207/12
Connections:
- new net N$43: 2N2.B, R19.1
- net CLK_IN: now also R19.2; no longer 2N2.B
Changed lines of the file:
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@@
 <part name="SUPPLY13" library="SparkFun-PowerSymbols" library_urn="urn:adsk.eagle:library:530" deviceset="5V" device=""/>
 <part name="C3" library="rcl" library_urn="urn:adsk.eagle:library:334" deviceset="CPOL-US" device="E2,5-6E" package3d_urn="urn:adsk.eagle:package:23430/1" value="100uf"/>
+<part name="R19" library="adafruit" library_urn="urn:adsk.eagle:library:420" deviceset="R-US_" device="0207/12" package3d_urn="urn:adsk.eagle:package:6240598/1" value="1K"/>
 </parts>
 <sheets>
@@
 <attribute name="VALUE" x="306.324" y="-59.309" size="1.778" layer="96" rot="R270"/>
 </instance>
+<instance part="R19" gate="G$1" x="185.42" y="-68.58" smashed="yes" rot="R180">
+<attribute name="VALUE" x="186.69" y="-70.358" size="1.778" layer="96" rot="R180"/>
+</instance>
 </instances>
 <busses>
@@
 </segment>
 <segment>
-<label x="187.96" y="-68.58" size="1.778" layer="95" rot="R180" xref="yes"/>
-<pinref part="2N2" gate="G$1" pin="B"/>
-<wire x1="187.96" y1="-68.58" x2="193.04" y2="-68.58" width="0.1524" layer="91"/>
+<label x="175.26" y="-68.58" size="1.778" layer="95" rot="R270" xref="yes"/>
+<wire x1="175.26" y1="-68.58" x2="180.34" y2="-68.58" width="0.1524" layer="91"/>
+<pinref part="R19" gate="G$1" pin="2"/>
 </segment>
 <segment>
@@
 </segment>
 </net>
+<net name="N$43" class="0">
+<segment>
+<pinref part="2N2" gate="G$1" pin="B"/>
+<wire x1="190.5" y1="-68.58" x2="193.04" y2="-68.58" width="0.1524" layer="91"/>
+<pinref part="R19" gate="G$1" pin="1"/>
+</segment>
+</net>
