File: modules/unipolar2bipolar/uni2bi.sch (EAGLE design)
At the start: 11 parts, among them IC1 LM324N

Commit message: uni2bi
Parts:
- removed R1, R2: 10k, adafruit:R-US_0207/10
- added R10, R9: 10k, adafruit:R-US_0207/10
Connections:
- net IN1 renamed UIN1
- net IN2 renamed UIN2
- removed net IN3: IC1C.+IN, JP2.5
- removed net IN4: IC1D.+IN, JP2.7
- removed net N$5: IC1D.OUT, R4.1
- removed net N$6: IC1C.OUT, R3.1
- removed net N$8: IC1A.OUT, R1.1
- removed net OUT1: IC1A.-IN, JP2.2, R1.2, R8.2
- removed net OUT2: IC1B.-IN, JP2.4, R2.2, R7.2
- removed net OUT3: IC1C.-IN, JP2.6, R3.2, R6.2
- removed net OUT4: IC1D.-IN, JP2.8, R4.2, R5.2
- new net BIN1: JP2.5, R4.1
- new net BIN2: JP2.7, R5.1
- new net BOUT1: IC1A.-IN, JP2.2, R10.1, R8.2
- new net BOUT2: IC1B.-IN, JP2.4, R6.1, R7.2
- new net N$1: IC1C.+IN, R4.2, R9.2
- new net N$2: IC1D.+IN, R3.2, R5.2
- new net N$4: IC1A.OUT, R10.2
- new net UOUT1: IC1C.-IN, IC1C.OUT, JP2.6
- new net UOUT2: IC1D.-IN, IC1D.OUT, JP2.8
- net +5V: now also R3.1, R9.1; no longer R5.1, R6.1
- net N$7: now also R6.2; no longer R2.1
Other:
- moved on the sheet: JP1, JP2
