File: modules/unipolar2bipolar/uni2bi.brd (EAGLE design)
At the start: 100 x 80 mm, 11 parts, among them IC1 LM324N

Commit message: uni2bi
Parts:
- removed R2: 10k, adafruit:0207/10
- added R9: 10k, adafruit:0207/10
- moved JP1 31.9 mm to (59.7, 34.3)
- moved R4 7.62 mm to (48.3, 20.3), turned to 90 degrees
- moved R3 5.08 mm to (55.9, 20.3), turned to 90 degrees
- moved R6 2.54 mm to (45.7, 20.3), turned to 90 degrees
- turned R10 to 90 degrees
- turned R5 to 90 degrees
- renumbered R1 to R10
Connections:
- net IN1 renamed UIN1
- net IN2 renamed UIN2
- removed net IN3: IC1.10, JP2.5
- removed net IN4: IC1.12, JP2.7
- removed net N$5: IC1.14, R4.1
- removed net N$6: IC1.8, R3.1
- removed net N$8: IC1.1, R10.1
- removed net OUT1: IC1.2, JP2.2, R10.2, R8.2
- removed net OUT2: IC1.6, JP2.4, R2.2, R7.2
- removed net OUT3: IC1.9, JP2.6, R3.2, R6.2
- removed net OUT4: IC1.13, JP2.8, R4.2, R5.2
- new net BIN1: JP2.5, R4.1
- new net BIN2: JP2.7, R5.1
- new net BOUT1: IC1.2, JP2.2, R10.1, R8.2
- new net BOUT2: IC1.6, JP2.4, R6.1, R7.2
- new net N$1: IC1.10, R4.2, R9.2
- new net N$2: IC1.12, R3.2, R5.2
- new net N$4: IC1.1, R10.2
- new net UOUT1: IC1.8, IC1.9, JP2.6
- new net UOUT2: IC1.13, IC1.14, JP2.8
- net +5V: now also R3.1, R9.1; no longer R5.1, R6.1
- net N$7: now also R6.2; no longer R2.1
Routing:
- net UOUT2: track 0.00 -> 54.7 mm
- net OUT2: track 34.8 -> 0.00 mm
- net N$5: track 33.0 -> 0.00 mm
- net BOUT2: track 0.00 -> 31.5 mm, vias 0 -> 1
- net N$2: track 0.00 -> 30.8 mm
- net OUT1: track 29.0 -> 0.00 mm
- net UOUT1: track 0.00 -> 28.2 mm
- net BOUT1: track 0.00 -> 26.7 mm
- net +12V: track 0.00 -> 25.4 mm
- net N$1: track 0.00 -> 22.4 mm
- net +5V: track 25.4 -> 47.3 mm
- net UIN2: track 0.00 -> 19.9 mm
- net UIN1: track 0.00 -> 19.1 mm
- net N$6: track 18.8 -> 0.00 mm
- net -12V: track 0.00 -> 16.8 mm
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Other:
- board size 100 x 80 mm -> 31.4 x 31.7 mm
- board text added: "+12"
- board text added: "+5"
- board text added: "-12"

Commit message: adsr board
Parts:
- moved JP1 2.54 mm to (59.7, 31.8)
Routing:
- net UOUT2: track 54.7 -> 43.5 mm, vias 0 -> 2
- net +5V: track 47.3 -> 42.7 mm
- net +12V: track 25.4 -> 28.7 mm
- net -12V: track 16.8 -> 19.4 mm
- net N$1: track 22.4 -> 20.9 mm
- net N$2: track 30.8 -> 30.0 mm
- net BOUT1: track 26.7 -> 25.9 mm
Other:
- board size 31.4 x 31.7 mm -> 27.6 x 30.5 mm
Changed lines of the file:
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@@
 <?xml version="1.0" encoding="utf-8"?>
 <!DOCTYPE eagle SYSTEM "eagle.dtd">
-<eagle version="9.6.2">
+<eagle version="9.5.2">
 <drawing>
 <settings>
@@
 <board>
 <plain>
-<wire x1="31.75" y1="8.89" x2="63.17" y2="8.89" width="0" layer="20"/>
-<wire x1="63.17" y1="8.89" x2="63.17" y2="40.63" width="0" layer="20"/>
-<wire x1="63.17" y1="40.63" x2="31.75" y2="40.63" width="0" layer="20"/>
-<wire x1="31.75" y1="40.63" x2="31.75" y2="8.89" width="0" layer="20"/>
-<hole x="35.56" y="36.83" drill="4.000246875"/>
-<hole x="59.69" y="16.51" drill="4.000246875"/>
-<text x="60.96" y="26.67" size="1.778" layer="26" rot="MR0">+5</text>
-<text x="57.15" y="31.75" size="1.778" layer="26" rot="MR0">+12</text>
-<text x="54.61" y="35.56" size="1.778" layer="26" rot="MR180">-12</text>
+<wire x1="35.56" y1="10.16" x2="63.17" y2="10.16" width="0" layer="20"/>
+<wire x1="63.17" y1="10.16" x2="63.17" y2="40.63" width="0" layer="20"/>
+<wire x1="63.17" y1="40.63" x2="35.56" y2="40.63" width="0" layer="20"/>
+<wire x1="35.56" y1="40.63" x2="35.56" y2="10.16" width="0" layer="20"/>
+<hole x="59.69" y="12.7" drill="4.000246875"/>
+<hole x="59.69" y="20.32" drill="4.000246875"/>
+<text x="60.96" y="24.13" size="1.778" layer="26" rot="MR0">+5</text>
+<text x="58.42" y="30.48" size="1.778" layer="26" rot="MR0">+12</text>
+<text x="54.61" y="34.29" size="1.778" layer="26" rot="MR180">-12</text>
 </plain>
 <attributes>
@@
 <attribute name="VALUE" x="40.259" y="32.385" size="1.27" layer="27" ratio="10"/>
 </element>
-<element name="JP1" library="pinhead" library_urn="urn:adsk.eagle:library:325" package="1X04" package3d_urn="urn:adsk.eagle:package:22407/2" value="" x="59.69" y="34.29" smashed="yes" rot="R90">
-<attribute name="POPULARITY" value="91" x="80.01" y="53.34" size="1.778" layer="27" rot="R90" display="off"/>
-<attribute name="VALUE" x="62.865" y="29.21" size="1.27" layer="27" rot="R90"/>
+<element name="JP1" library="pinhead" library_urn="urn:adsk.eagle:library:325" package="1X04" package3d_urn="urn:adsk.eagle:package:22407/2" value="" x="59.69" y="31.75" smashed="yes" rot="R90">
+<attribute name="POPULARITY" value="91" x="80.01" y="50.8" size="1.778" layer="27" rot="R90" display="off"/>
+<attribute name="VALUE" x="62.865" y="26.67" size="1.27" layer="27" rot="R90"/>
 </element>
 <element name="JP2" library="pinhead" library_urn="urn:adsk.eagle:library:325" package="1X08" package3d_urn="urn:adsk.eagle:package:22409/2" value="" x="46.99" y="12.7" smashed="yes">
@@
 <contactref element="R8" pad="2"/>
 <contactref element="IC1" pad="2"/>
-<wire x1="36.83" y1="15.24" x2="38.1" y2="15.24" width="0.1524" layer="1"/>
+<wire x1="36.83" y1="16.51" x2="38.1" y2="15.24" width="0.1524" layer="1"/>
 <contactref element="R10" pad="1"/>
 <wire x1="38.1" y1="15.24" x2="40.64" y2="15.24" width="0.1524" layer="1"/>
@@
 <wire x1="38.7223625" y1="30.48" x2="38.1" y2="30.48" width="0.1524" layer="1"/>
 <wire x1="38.1" y1="30.48" x2="36.83" y2="29.21" width="0.1524" layer="1"/>
-<wire x1="36.83" y1="29.21" x2="36.83" y2="15.24" width="0.1524" layer="1"/>
+<wire x1="36.83" y1="29.21" x2="36.83" y2="16.51" width="0.1524" layer="1"/>
 <wire x1="41.91" y1="29.21" x2="40.3606" y2="30.7594" width="0.1524" layer="1"/>
 <wire x1="40.3606" y1="30.7594" x2="39.0017625" y2="30.7594" width="0.1524" layer="1"/>
@@
 <contactref element="JP2" pad="8"/>
 <contactref element="IC1" pad="13"/>
-<wire x1="41.91" y1="36.83" x2="39.37" y2="34.29" width="0.1524" layer="1"/>
-<wire x1="39.37" y1="34.29" x2="38.1" y2="34.29" width="0.1524" layer="1"/>
-<wire x1="38.1" y1="34.29" x2="35.56" y2="31.75" width="0.1524" layer="1"/>
-<wire x1="35.56" y1="31.75" x2="35.56" y2="10.16" width="0.1524" layer="1"/>
-<wire x1="35.56" y1="10.16" x2="54.61" y2="10.16" width="0.1524" layer="1"/>
-<wire x1="54.61" y1="10.16" x2="55.88" y2="11.43" width="0.1524" layer="1"/>
-<wire x1="55.88" y1="11.43" x2="55.88" y2="12.7" width="0.1524" layer="1"/>
 <contactref element="IC1" pad="14"/>
 <wire x1="41.91" y1="36.83" x2="39.37" y2="36.83" width="0.1524" layer="1"/>
+<wire x1="41.91" y1="36.83" x2="41.91" y2="34.29" width="0.1524" layer="16"/>
+<wire x1="41.91" y1="34.29" x2="40.64" y2="33.02" width="0.1524" layer="16"/>
+<wire x1="40.64" y1="33.02" x2="40.64" y2="27.94" width="0.1524" layer="16"/>
+<wire x1="40.64" y1="27.94" x2="39.37" y2="26.67" width="0.1524" layer="16"/>
+<wire x1="39.37" y1="26.67" x2="39.37" y2="19.05" width="0.1524" layer="16"/>
+<via x="39.37" y="19.05" extent="1-16" drill="0.35"/>
+<wire x1="39.37" y1="19.05" x2="54.61" y2="19.05" width="0.1524" layer="1"/>
+<via x="54.61" y="19.05" extent="1-16" drill="0.35"/>
+<wire x1="54.61" y1="13.97" x2="55.88" y2="12.7" width="0.1524" layer="16"/>
+<wire x1="54.61" y1="19.05" x2="54.61" y2="13.97" width="0.1524" layer="16"/>
 </signal>
 <signal name="+12V">
@@
 <wire x1="48.26" y1="33.02" x2="48.26" y2="38.1" width="0.1524" layer="16"/>
 <wire x1="48.26" y1="38.1" x2="48.5394" y2="38.3794" width="0.1524" layer="16"/>
-<wire x1="55.6006" y1="38.3794" x2="57.15" y2="36.83" width="0.1524" layer="16"/>
+<wire x1="55.6006" y1="38.3794" x2="55.88" y2="38.1" width="0.1524" layer="16"/>
 <wire x1="48.5394" y1="38.3794" x2="55.6006" y2="38.3794" width="0.1524" layer="16"/>
-<wire x1="57.15" y1="36.83" x2="57.15" y2="33.02" width="0.1524" layer="16"/>
-<wire x1="57.15" y1="33.02" x2="59.69" y2="33.02" width="0.1524" layer="16"/>
+<wire x1="55.88" y1="38.1" x2="55.88" y2="30.48" width="0.1524" layer="16"/>
+<wire x1="55.88" y1="30.48" x2="59.69" y2="30.48" width="0.1524" layer="16"/>
 </signal>
 <signal name="-12V">
@@
 <contactref element="IC1" pad="11"/>
 <wire x1="46.99" y1="36.83" x2="46.99" y2="39.37" width="0.1524" layer="16"/>
-<wire x1="55.88" y1="39.37" x2="59.69" y2="35.56" width="0.1524" layer="16"/>
+<wire x1="59.69" y1="33.02" x2="57.15" y2="35.56" width="0.1524" layer="16"/>
+<wire x1="57.15" y1="38.1" x2="57.15" y2="35.56" width="0.1524" layer="16"/>
+<wire x1="57.15" y1="38.1" x2="55.88" y2="39.37" width="0.1524" layer="16"/>
 <wire x1="46.99" y1="39.37" x2="55.88" y2="39.37" width="0.1524" layer="16"/>
 </signal>
@@
 <contactref element="R7" pad="1"/>
 <wire x1="57.15" y1="22.86" x2="55.88" y2="22.86" width="0.1524" layer="1"/>
-<wire x1="55.88" y1="22.86" x2="43.18" y2="22.86" width="0.1524" layer="1"/>
-<wire x1="43.18" y1="22.86" x2="38.1" y2="22.86" width="0.1524" layer="1"/>
-<wire x1="38.1" y1="22.86" x2="38.1" y2="25.4" width="0.1524" layer="1"/>
-<wire x1="43.18" y1="25.4" x2="43.18" y2="22.86" width="0.1524" layer="1"/>
-<wire x1="59.69" y1="30.48" x2="59.69" y2="25.4" width="0.1524" layer="1"/>
+<wire x1="55.88" y1="24.13" x2="43.18" y2="24.13" width="0.1524" layer="1"/>
+<wire x1="43.18" y1="24.13" x2="39.37" y2="24.13" width="0.1524" layer="1"/>
+<wire x1="39.37" y1="24.13" x2="38.1" y2="25.4" width="0.1524" layer="1"/>
+<wire x1="43.18" y1="25.4" x2="43.18" y2="24.13" width="0.1524" layer="1"/>
+<wire x1="59.69" y1="27.94" x2="59.69" y2="25.4" width="0.1524" layer="1"/>
 <wire x1="59.69" y1="25.4" x2="57.15" y2="22.86" width="0.1524" layer="1"/>
 <contactref element="R9" pad="1"/>
@@
 <wire x1="54.61" y1="16.51" x2="55.88" y2="15.24" width="0.1524" layer="1"/>
 <wire x1="55.88" y1="15.24" x2="55.88" y2="22.86" width="0.1524" layer="1"/>
+<wire x1="55.88" y1="22.86" x2="55.88" y2="24.13" width="0.1524" layer="1"/>
 </signal>
 <signal name="GND">
@@
 <wire x1="52.4382375" y1="27.6606" x2="52.7176375" y2="27.94" width="0.1524" layer="1"/>
 <wire x1="52.7176375" y1="27.94" x2="53.34" y2="27.94" width="0.1524" layer="1"/>
-<wire x1="48.26" y1="27.6606" x2="52.4382375" y2="27.6606" width="0.1524" layer="1"/>
+<wire x1="47.9806" y1="27.6606" x2="52.4382375" y2="27.6606" width="0.1524" layer="1"/>
 <wire x1="53.34" y1="27.94" x2="54.61" y2="29.21" width="0.1524" layer="1"/>
 <contactref element="R6" pad="2"/>
 <wire x1="45.72" y1="25.4" x2="47.9806" y2="27.6606" width="0.1524" layer="1"/>
-<wire x1="47.9806" y1="27.6606" x2="48.26" y2="27.6606" width="0.1524" layer="1"/>
 </signal>
 <signal name="N$1">
@@
 <wire x1="50.8" y1="25.4" x2="52.07" y2="26.67" width="0.1524" layer="1"/>
 <wire x1="54.61" y1="26.67" x2="55.88" y2="27.94" width="0.1524" layer="1"/>
-<wire x1="55.88" y1="27.94" x2="55.88" y2="33.02" width="0.1524" layer="1"/>
-<wire x1="55.88" y1="33.02" x2="54.61" y2="34.29" width="0.1524" layer="1"/>
-<wire x1="54.61" y1="34.29" x2="50.8" y2="34.29" width="0.1524" layer="1"/>
+<wire x1="55.88" y1="27.94" x2="55.88" y2="30.48" width="0.1524" layer="1"/>
+<wire x1="55.88" y1="30.48" x2="52.07" y2="34.29" width="0.1524" layer="1"/>
+<wire x1="52.07" y1="34.29" x2="50.8" y2="34.29" width="0.1524" layer="1"/>
 <wire x1="50.8" y1="34.29" x2="49.53" y2="35.56" width="0.1524" layer="1"/>
 <wire x1="49.53" y1="35.56" x2="49.53" y2="36.83" width="0.1524" layer="1"/>
@@
 <wire x1="53.34" y1="25.4" x2="55.88" y2="25.4" width="0.1524" layer="1"/>
 <wire x1="55.88" y1="25.4" x2="57.15" y2="26.67" width="0.1524" layer="1"/>
-<wire x1="57.15" y1="26.67" x2="57.15" y2="38.1" width="0.1524" layer="1"/>
-<wire x1="57.15" y1="38.1" x2="55.88" y2="39.37" width="0.1524" layer="1"/>
-<wire x1="55.88" y1="39.37" x2="45.72" y2="39.37" width="0.1524" layer="1"/>
+<wire x1="57.15" y1="26.67" x2="57.15" y2="36.83" width="0.1524" layer="1"/>
+<wire x1="57.15" y1="36.83" x2="54.61" y2="39.37" width="0.1524" layer="1"/>
+<wire x1="54.61" y1="39.37" x2="45.72" y2="39.37" width="0.1524" layer="1"/>
 <wire x1="45.72" y1="39.37" x2="44.45" y2="38.1" width="0.1524" layer="1"/>
 <wire x1="44.45" y1="38.1" x2="44.45" y2="36.83" width="0.1524" layer="1"/>
