File: modules/midi2cv/circuit/midi2cv.brd (EAGLE design)
At the start: 56.8 x 63.5 mm, 17 parts, among them U1 MICROCHIP_MCP4902-E-PMICROCHI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, U2 MICROCHIP_MCP4902-E-PMICROCHI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, U3 MICROCHIP_MCP4902-E-PMICROCHI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

Commit message: midi2cv board
Parts:
- moved D1 13.3 mm to (72.4, 12.7)
- moved OK1 12.0 mm to (58.4, 15.2)
- moved 12BITDAC1 8.03 mm to (57.1, 30.5)
- moved U3 7.62 mm to (57.1, 49.5)
- moved FTDI 4.58 mm to (83.8, 57.1)
- moved 12BITDAC 2.54 mm to (72.4, 22.9)
Connections:
- net CS4: now also U3.3; no longer U1.3
- net CS5: now also U1.3; no longer U2.3
- net CS6: now also U2.3; no longer U3.3

Commit message: midi2cv
Parts:
- moved JP1 65.7 mm to (40.6, 45.7), turned to 90 degrees
- moved DIN5 65.4 mm to (40.6, 59.7), turned to 90 degrees
- moved D1 55.1 mm to (48.3, 62.2)
- moved R3 54.5 mm to (59.7, 62.2)
- moved R2 53.2 mm to (50.8, 50.8), turned to 270 degrees
- moved R4 49.8 mm to (80.0, 57.1)
- moved C1 43.5 mm to (90.2, 57.1), turned to 180 degrees
- moved OK1 40.6 mm to (58.4, 55.9), turned to 90 degrees
- moved JP2 22.2 mm to (41.9, 21.6), turned to 90 degrees
- moved 12BITDAC1 15.3 mm to (58.4, 15.2), turned to 270 degrees
- moved U3 10.2 mm to (58.4, 39.4)
- moved 12BITDAC 7.73 mm to (71.1, 15.2), turned to 270 degrees
- moved 12BITDAC2 7.73 mm to (86.4, 15.2), turned to 270 degrees
- moved FTDI 4.02 mm to (85.1, 61.0)
- moved U1 2.54 mm to (85.1, 39.4)
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Connections:
- net +5V: now also U1.9, U2.9, U3.9
Routing:
- net GND: track 0.00 -> 295.8 mm, vias 0 -> 1
- net +5V: track 0.00 -> 221.2 mm
- net MOSI: track 0.00 -> 133.2 mm
- net SCK: track 0.00 -> 106.3 mm
- net CS1: track 0.00 -> 96.4 mm
- net CS2: track 0.00 -> 85.0 mm, vias 0 -> 1
- net PITCH_CV3: track 0.00 -> 84.6 mm
- net CS3: track 0.00 -> 78.9 mm, vias 0 -> 1
- net CC2: track 0.00 -> 75.2 mm, vias 0 -> 1
- net LEVEL2: track 0.00 -> 70.2 mm
- net CS4: track 0.00 -> 57.3 mm, vias 0 -> 2
- net CC3: track 0.00 -> 56.8 mm
- net TX: track 0.00 -> 53.8 mm
- net LEVEL3: track 0.00 -> 52.5 mm, vias 0 -> 1
- net RX: track 0.00 -> 44.3 mm
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Other:
- board size 56.8 x 63.5 mm -> 65.7 x 64.8 mm

Commit message: midi2cv
Parts:
- moved JP1 1.27 mm to (41.9, 45.7)
Routing:
- net CC2: track 75.2 -> 73.2 mm
- net CLOCK_OUT: track 7.40 -> 6.13 mm
- net CC3: track 56.8 -> 58.1 mm
- net CC1: track 27.5 -> 26.2 mm
- net GATE3: track 16.9 -> 16.3 mm
- net GATE2: track 16.9 -> 16.3 mm
Other:
- board text added: "2"
- board text added: "4"
- board text added: "5"
- board text added: "C1"
- board text added: "C2"
- board text added: "C3"
- board text added: "CK"
- board text added: "G1"
- board text added: "G2"
- board text added: "G3"
- board text added: "GND"
- board text added: "L1"
- board text added: "L2"
- board text added: "L3"
- board text added: "P1"
- board text added: "P2"
- board text added: "P3"
Changed lines of the file:
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@@
 <?xml version="1.0" encoding="utf-8"?>
 <!DOCTYPE eagle SYSTEM "eagle.dtd">
-<eagle version="9.6.2">
+<eagle version="9.5.2">
 <drawing>
 <settings>
@@
 <wire x1="102.54" y1="64.76" x2="36.83" y2="64.76" width="0" layer="20"/>
 <wire x1="36.83" y1="64.76" x2="36.83" y2="0" width="0" layer="20"/>
+<text x="36.83" y="12.7" size="1.778" layer="21">P1</text>
+<text x="36.83" y="15.24" size="1.778" layer="21">P2</text>
+<text x="36.83" y="17.78" size="1.778" layer="21">P3</text>
+<text x="36.83" y="20.32" size="1.778" layer="21">L1</text>
+<text x="36.83" y="22.86" size="1.778" layer="21">L2</text>
+<text x="36.83" y="25.4" size="1.778" layer="21">L3</text>
+<text x="36.83" y="27.94" size="1.778" layer="21">G1</text>
+<text x="36.83" y="36.83" size="1.778" layer="21">G2</text>
+<text x="36.83" y="39.37" size="1.778" layer="21">G3</text>
+<text x="36.83" y="41.91" size="1.778" layer="21">C1</text>
+<text x="36.83" y="44.45" size="1.778" layer="21">C2</text>
+<text x="36.83" y="46.99" size="1.778" layer="21">C3</text>
+<text x="36.83" y="49.53" size="1.778" layer="21">CK</text>
+<text x="36.83" y="60.96" size="1.778" layer="21">5</text>
+<text x="36.83" y="55.88" size="1.778" layer="21">4</text>
+<text x="36.83" y="58.42" size="1.778" layer="21">2</text>
+<text x="74.93" y="62.23" size="1.778" layer="21">GND</text>
 </plain>
 <attributes>
@@
 </element>
 <element name="FTDI" library="pinhead" library_urn="urn:adsk.eagle:library:325" package="1X06" package3d_urn="urn:adsk.eagle:package:22472/2" value="" x="85.09" y="60.96" smashed="yes">
-<attribute name="NAME" x="77.3938" y="62.7888" size="1.27" layer="25" ratio="10"/>
+<attribute name="NAME" x="86.2838" y="62.7888" size="1.27" layer="25" ratio="10"/>
 <attribute name="POPULARITY" value="79" x="85.09" y="60.96" size="1.778" layer="27" display="off"/>
 <attribute name="VALUE" x="77.47" y="57.785" size="1.27" layer="27"/>
 </element>
-<element name="JP1" library="pinhead" library_urn="urn:adsk.eagle:library:325" package="1X07" package3d_urn="urn:adsk.eagle:package:22477/2" value="" x="40.64" y="45.72" smashed="yes" rot="R90">
-<attribute name="NAME" x="38.8112" y="36.7538" size="1.27" layer="25" ratio="10" rot="R90"/>
-<attribute name="POPULARITY" value="0" x="40.64" y="45.72" size="1.778" layer="27" rot="R90" display="off"/>
-<attribute name="VALUE" x="43.815" y="36.83" size="1.27" layer="27" rot="R90"/>
+<element name="JP1" library="pinhead" library_urn="urn:adsk.eagle:library:325" package="1X07" package3d_urn="urn:adsk.eagle:package:22477/2" value="" x="41.91" y="45.72" smashed="yes" rot="R90">
+<attribute name="POPULARITY" value="0" x="41.91" y="45.72" size="1.778" layer="27" rot="R90" display="off"/>
+<attribute name="VALUE" x="45.085" y="36.83" size="1.27" layer="27" rot="R90"/>
 </element>
 <element name="JP2" library="pinhead" library_urn="urn:adsk.eagle:library:325" package="1X07" package3d_urn="urn:adsk.eagle:package:22477/2" value="" x="41.91" y="21.59" smashed="yes" rot="R90">
-<attribute name="NAME" x="40.0812" y="12.6238" size="1.27" layer="25" ratio="10" rot="R90"/>
 <attribute name="POPULARITY" value="0" x="41.91" y="21.59" size="1.778" layer="27" rot="R90" display="off"/>
 <attribute name="VALUE" x="45.085" y="12.7" size="1.27" layer="27" rot="R90"/>
 </element>
 <element name="DIN5" library="pinhead" library_urn="urn:adsk.eagle:library:325" package="1X03" package3d_urn="urn:adsk.eagle:package:22458/2" value="" x="40.64" y="59.69" smashed="yes" rot="R90">
-<attribute name="NAME" x="38.8112" y="55.8038" size="1.27" layer="25" ratio="10" rot="R90"/>
 <attribute name="POPULARITY" value="92" x="40.64" y="59.69" size="1.778" layer="27" rot="R90" display="off"/>
 <attribute name="VALUE" x="43.815" y="55.88" size="1.27" layer="27" rot="R90"/>
@@
 <contactref element="B1" pad="D3"/>
 <contactref element="JP1" pad="6"/>
-<wire x1="40.64" y1="50.8" x2="44.45" y2="50.8" width="0.1524" layer="1"/>
+<wire x1="41.91" y1="50.8" x2="44.45" y2="50.8" width="0.1524" layer="1"/>
 <wire x1="44.45" y1="50.8" x2="46.99" y2="48.26" width="0.1524" layer="1"/>
 </signal>
@@
 <contactref element="JP1" pad="3"/>
 <wire x1="60.96" y1="35.56" x2="62.23" y2="36.83" width="0.1524" layer="1"/>
-<wire x1="40.64" y1="43.18" x2="41.91" y2="43.18" width="0.1524" layer="1"/>
 <wire x1="41.91" y1="43.18" x2="44.45" y2="40.64" width="0.1524" layer="1"/>
 <wire x1="44.45" y1="40.64" x2="44.45" y2="36.83" width="0.1524" layer="1"/>
@@
 <via x="52.07" y="26.67" extent="1-16" drill="0.35"/>
 <wire x1="52.07" y1="35.56" x2="52.07" y2="26.67" width="0.1524" layer="16"/>
-<wire x1="52.07" y1="35.56" x2="44.45" y2="35.56" width="0.1524" layer="16"/>
-<wire x1="44.45" y1="35.56" x2="44.45" y2="43.18" width="0.1524" layer="16"/>
-<wire x1="44.45" y1="43.18" x2="41.91" y2="45.72" width="0.1524" layer="16"/>
-<wire x1="41.91" y1="45.72" x2="40.64" y2="45.72" width="0.1524" layer="16"/>
+<wire x1="52.07" y1="35.56" x2="45.72" y2="35.56" width="0.1524" layer="16"/>
+<wire x1="45.72" y1="35.56" x2="45.72" y2="41.91" width="0.1524" layer="16"/>
+<wire x1="45.72" y1="41.91" x2="41.91" y2="45.72" width="0.1524" layer="16"/>
 </signal>
 <signal name="LEVEL3">
@@
 <contactref element="JP1" pad="5"/>
 <wire x1="39.37" y1="48.26" x2="38.1" y2="46.99" width="0.1524" layer="1"/>
-<wire x1="39.37" y1="48.26" x2="40.64" y2="48.26" width="0.1524" layer="1"/>
+<wire x1="39.37" y1="48.26" x2="41.91" y2="48.26" width="0.1524" layer="1"/>
 <wire x1="38.1" y1="33.02" x2="38.2524" y2="32.8676" width="0.1524" layer="1"/>
 <wire x1="38.2524" y1="32.8676" x2="72.2376" y2="32.8676" width="0.1524" layer="1"/>
@@
 <contactref element="B1" pad="D12"/>
 <contactref element="JP1" pad="1"/>
-<wire x1="43.6626" y1="32.5374" x2="40.64" y2="35.56" width="0.1524" layer="16"/>
-<wire x1="40.64" y1="35.56" x2="40.64" y2="38.1" width="0.1524" layer="16"/>
+<wire x1="43.6626" y1="32.5374" x2="41.91" y2="34.29" width="0.1524" layer="16"/>
+<wire x1="41.91" y1="34.29" x2="41.91" y2="38.1" width="0.1524" layer="16"/>
 <wire x1="46.99" y1="23.876" x2="43.6626" y2="27.2034" width="0.1524" layer="16"/>
 <wire x1="43.6626" y1="27.2034" x2="43.6626" y2="32.5374" width="0.1524" layer="16"/>
@@
 <contactref element="B1" pad="D11"/>
 <contactref element="JP1" pad="2"/>
-<wire x1="43.18" y1="38.1" x2="43.18" y2="35.56" width="0.1524" layer="16"/>
-<wire x1="43.18" y1="35.56" x2="44.45" y2="34.29" width="0.1524" layer="16"/>
 <wire x1="44.45" y1="28.956" x2="46.99" y2="26.416" width="0.1524" layer="16"/>
-<wire x1="40.64" y1="40.64" x2="43.18" y2="38.1" width="0.1524" layer="16"/>
-<wire x1="44.45" y1="34.29" x2="44.45" y2="28.956" width="0.1524" layer="16"/>
+<wire x1="41.91" y1="40.64" x2="44.45" y2="38.1" width="0.1524" layer="16"/>
+<wire x1="44.45" y1="38.1" x2="44.45" y2="28.956" width="0.1524" layer="16"/>
 </signal>
 <signal name="GND">
