File: modules/midi2cv/circuit/midi2cv.sch (EAGLE design)
At the start: 17 parts, among them U1 MICROCHIP_MCP4902-E-PMICROCHI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, U2 MICROCHIP_MCP4902-E-PMICROCHI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, U3 MICROCHIP_MCP4902-E-PMICROCHI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

Commit message: midi2cv board
Connections:
- net CS4: now also U3.!CS!; no longer U1.!CS!
- net CS5: now also U1.!CS!; no longer U2.!CS!
- net CS6: now also U2.!CS!; no longer U3.!CS!
Changed lines of the file:
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@@
 <?xml version="1.0" encoding="utf-8"?>
 <!DOCTYPE eagle SYSTEM "eagle.dtd">
-<eagle version="9.6.2">
+<eagle version="9.5.2">
 <drawing>
 <settings>
@@
 </segment>
 <segment>
+<pinref part="U3" gate="G$0" pin="!CS!"/>
+<wire x1="81.28" y1="40.64" x2="78.74" y2="40.64" width="0.1524" layer="91"/>
+<label x="78.74" y="40.64" size="1.778" layer="95" rot="R180" xref="yes"/>
+</segment>
+</net>
+<net name="CS5" class="0">
+<segment>
+<pinref part="B1" gate="G$1" pin="A4"/>
+<wire x1="-33.02" y1="116.84" x2="-35.56" y2="116.84" width="0.1524" layer="91"/>
+<label x="-35.56" y="116.84" size="1.778" layer="95" rot="R180" xref="yes"/>
+</segment>
+<segment>
 <pinref part="U1" gate="G$0" pin="!CS!"/>
 <wire x1="157.48" y1="40.64" x2="154.94" y2="40.64" width="0.1524" layer="91"/>
@@
 </segment>
 </net>
-<net name="CS5" class="0">
-<segment>
-<pinref part="B1" gate="G$1" pin="A4"/>
-<wire x1="-33.02" y1="116.84" x2="-35.56" y2="116.84" width="0.1524" layer="91"/>
-<label x="-35.56" y="116.84" size="1.778" layer="95" rot="R180" xref="yes"/>
+<net name="CS6" class="0">
+<segment>
+<pinref part="B1" gate="G$1" pin="A5"/>
+<wire x1="-33.02" y1="114.3" x2="-43.18" y2="114.3" width="0.1524" layer="91"/>
+<label x="-43.18" y="114.3" size="1.778" layer="95" rot="R180" xref="yes"/>
 </segment>
 <segment>
@@
 </segment>
 </net>
-<net name="CS6" class="0">
-<segment>
-<pinref part="B1" gate="G$1" pin="A5"/>
-<wire x1="-33.02" y1="114.3" x2="-43.18" y2="114.3" width="0.1524" layer="91"/>
-<label x="-43.18" y="114.3" size="1.778" layer="95" rot="R180" xref="yes"/>
-</segment>
-<segment>
-<pinref part="U3" gate="G$0" pin="!CS!"/>
-<wire x1="81.28" y1="40.64" x2="78.74" y2="40.64" width="0.1524" layer="91"/>
-<label x="78.74" y="40.64" size="1.778" layer="95" rot="R180" xref="yes"/>
-</segment>
-</net>

Commit message: midi2cv
Connections:
- net +5V: now also U1.!SHDN!, U2.!SHDN!, U3.!SHDN!
Changed lines of the file:
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@@
 <?xml version="1.0" encoding="utf-8"?>
 <!DOCTYPE eagle SYSTEM "eagle.dtd">
-<eagle version="9.5.2">
+<eagle version="9.6.2">
 <drawing>
 <settings>
@@
 <pinref part="P+7" gate="1" pin="+5V"/>
 <wire x1="76.2" y1="22.86" x2="68.58" y2="22.86" width="0.1524" layer="91"/>
+<pinref part="U3" gate="G$0" pin="!SHDN!"/>
+<wire x1="81.28" y1="30.48" x2="76.2" y2="30.48" width="0.1524" layer="91"/>
+<wire x1="76.2" y1="30.48" x2="76.2" y2="25.4" width="0.1524" layer="91"/>
+<junction x="76.2" y="25.4"/>
 </segment>
 <segment>
@@
 <pinref part="P+6" gate="1" pin="+5V"/>
 <wire x1="152.4" y1="22.86" x2="147.32" y2="22.86" width="0.1524" layer="91"/>
+<pinref part="U1" gate="G$0" pin="!SHDN!"/>
+<wire x1="157.48" y1="30.48" x2="152.4" y2="30.48" width="0.1524" layer="91"/>
+<wire x1="152.4" y1="30.48" x2="152.4" y2="25.4" width="0.1524" layer="91"/>
+<junction x="152.4" y="25.4"/>
 </segment>
 <segment>
@@
 <pinref part="P+5" gate="1" pin="+5V"/>
 <wire x1="236.22" y1="22.86" x2="228.6" y2="22.86" width="0.1524" layer="91"/>
-</segment>
-<segment>
+<pinref part="U2" gate="G$0" pin="!SHDN!"/>
+<wire x1="243.84" y1="30.48" x2="236.22" y2="30.48" width="0.1524" layer="91"/>
+<wire x1="236.22" y1="30.48" x2="236.22" y2="25.4" width="0.1524" layer="91"/>
+<junction x="236.22" y="25.4"/>
+</segment>
+<segment>
