File: modules/adsr/circuit/adsr.sch (EAGLE design)
At the start: 5 parts, among them U1 ARDUINO_PRO_MINI

Commit message: adsr
Parts:
- removed ADSR_KNOB: (no value), pinhead:PINHD-1X4
- removed U1: ARDUINO_PRO_MINI, ARDUINO_PRO_MINI:ARDUINO_PRO_MINI
- added BLUE, GREEN, RED, YELLOW: (no value), SparkFun-LED:LED-5MM-KIT-NO-SILK
- added FUTURE: (no value), pinhead:PINHD-1X2
- added R1: 330, SparkFun-Resistors:330OHM-HORIZ-1/10W-5%
- added U$2: ARDUINO_MINI, SparkFun-Retired:ARDUINO_MINI
Connections:
- removed net N$1: U$1.SCK, U1.SCK
- removed net N$2: U$1.SDI, U1.MOSI
- new net AVSS: U$1.AVSS, U$1.LDAC
- new net CS: U$1.#CS, U$2.10
- new net MOSI: U$1.SDI, U$2.11
- new net N$10: FUTURE.1, U$2.9
- new net N$4: BLUE.C, U$2.7
- new net N$5: U$2.6, YELLOW.C
- new net N$6: GREEN.C, U$2.5
- new net N$7: RED.C, U$2.4
- new net N$8: BLUE.A, GREEN.A, R1.2, RED.A, YELLOW.A
- new net N$9: FUTURE.2, U$2.8
- new net SCK: U$1.SCK, U$2.13
- net +5V: now also R1.1, U$1.REFA, U$1.VDD, U$2.VCC
- net A: now also ADSR_CV.1, U$2.A0; no longer U1.A0
- net D: now also ADSR_CV.2, U$2.A1; no longer U1.A1
- net GATE_IN: now also U$2.3; no longer U1.D2
- net GND: now also U$2.GND, U$2.GND@2; no longer U$1.#CS
- net R: now also ADSR_CV.4, U$2.A3; no longer U1.A3
- net S: now also ADSR_CV.3, U$2.A2; no longer U1.A2
Other:
- moved on the sheet: ADSR_CV

Commit message: adsr
Connections:
- removed net AVSS: U$1.AVSS, U$1.LDAC
- net GND: now also U$1.AVSS, U$1.LDAC
Changed lines of the file:
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@@
 <part name="U$1" library="adafruit" library_urn="urn:adsk.eagle:library:420" deviceset="MCP4921" device="" package3d_urn="urn:adsk.eagle:package:6240674/1"/>
 <part name="SUPPLY1" library="supply2" library_urn="urn:adsk.eagle:library:372" deviceset="+5V" device=""/>
-<part name="SUPPLY2" library="supply2" library_urn="urn:adsk.eagle:library:372" deviceset="GND" device=""/>
 <part name="ADSR_CV" library="pinhead" library_urn="urn:adsk.eagle:library:325" deviceset="PINHD-1X4" device="" package3d_urn="urn:adsk.eagle:package:22407/2"/>
 <part name="JP3" library="pinhead" library_urn="urn:adsk.eagle:library:325" deviceset="PINHD-1X4" device="" package3d_urn="urn:adsk.eagle:package:22407/2"/>
@@
 <part name="SUPPLY8" library="supply2" library_urn="urn:adsk.eagle:library:372" deviceset="GND" device=""/>
 <part name="SUPPLY9" library="supply2" library_urn="urn:adsk.eagle:library:372" deviceset="GND" device=""/>
+<part name="SUPPLY2" library="supply2" library_urn="urn:adsk.eagle:library:372" deviceset="GND" device=""/>
 </parts>
 <sheets>
@@
 <attribute name="VALUE" x="114.935" y="64.135" size="1.778" layer="96"/>
 </instance>
-<instance part="SUPPLY2" gate="GND" x="2.54" y="-27.94" smashed="yes"/>
 <instance part="ADSR_CV" gate="A" x="132.08" y="76.2" smashed="yes">
 <attribute name="NAME" x="125.73" y="84.455" size="1.778" layer="95"/>
@@
 <instance part="SUPPLY8" gate="GND" x="71.12" y="78.74" smashed="yes"/>
 <instance part="SUPPLY9" gate="GND" x="-33.02" y="73.66" smashed="yes"/>
+<instance part="SUPPLY2" gate="GND" x="2.54" y="-27.94" smashed="yes"/>
 </instances>
 <busses>
@@
 <wire x1="-33.02" y1="81.28" x2="-33.02" y2="76.2" width="0.1524" layer="91"/>
 <pinref part="SUPPLY9" gate="GND" pin="GND"/>
+</segment>
+<segment>
+<pinref part="U$1" gate="G$1" pin="LDAC"/>
+<wire x1="5.08" y1="-12.7" x2="2.54" y2="-12.7" width="0.1524" layer="91"/>
+<wire x1="2.54" y1="-12.7" x2="2.54" y2="-25.4" width="0.1524" layer="91"/>
+<pinref part="U$1" gate="G$1" pin="AVSS"/>
+<wire x1="20.32" y1="-25.4" x2="2.54" y2="-25.4" width="0.1524" layer="91"/>
+<pinref part="SUPPLY2" gate="GND" pin="GND"/>
+<junction x="2.54" y="-25.4"/>
 </segment>
 </net>
@@
 </segment>
 </net>
-<net name="AVSS" class="0">
-<segment>
-<pinref part="U$1" gate="G$1" pin="LDAC"/>
-<wire x1="5.08" y1="-12.7" x2="2.54" y2="-12.7" width="0.1524" layer="91"/>
-<pinref part="SUPPLY2" gate="GND" pin="GND"/>
-<wire x1="2.54" y1="-12.7" x2="2.54" y2="-25.4" width="0.1524" layer="91"/>
-<pinref part="U$1" gate="G$1" pin="AVSS"/>
-<wire x1="20.32" y1="-25.4" x2="2.54" y2="-25.4" width="0.1524" layer="91"/>
-<junction x="2.54" y="-25.4"/>
-</segment>
-</net>
