File: modules/osc/circuit/VCO-revb.brd (EAGLE design)
At the start: 84.8 x 45.7 mm, 25 parts, among them Q1 16MHZ

Commit message: vcf done
Connections:
- net 3.3V: no longer STATUS.A
- net VDD: now also STATUS.A
Routing:
- net VDD: track 97.2 -> 110.8 mm
- net 3.3V: track 221.8 -> 219.3 mm
Changed lines of the file:
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@@
 <?xml version="1.0" encoding="utf-8"?>
 <!DOCTYPE eagle SYSTEM "eagle.dtd">
-<eagle version="9.5.2">
+<eagle version="9.6.2">
 <drawing>
 <settings>
@@
 <attribute name="POPULARITY" value="56" x="34.29" y="39.37" size="1.778" layer="27" rot="R180" display="off"/>
 <attribute name="SPICEPREFIX" value="C" x="34.29" y="39.37" size="1.778" layer="27" rot="R180" display="off"/>
-<attribute name="VALUE" x="37.338" y="38.227" size="1.27" layer="27" ratio="10" rot="R180"/>
+<attribute name="VALUE" x="36.068" y="42.037" size="1.27" layer="27" ratio="10" rot="R180"/>
 </element>
 <element name="C5" library="rcl" library_urn="urn:adsk.eagle:library:334" package="C025-024X044" package3d_urn="urn:adsk.eagle:package:23630/1" value="01uf" x="3.81" y="30.48" smashed="yes" rot="R180">
@@
 <contactref element="C1" pad="2"/>
 <wire x1="29.21" y1="13.97" x2="31.75" y2="16.51" width="0.1524" layer="16"/>
+<contactref element="STATUS" pad="A"/>
+<wire x1="22.86" y1="3.81" x2="22.86" y2="5.08" width="0.1524" layer="1"/>
+<wire x1="22.86" y1="5.08" x2="26.67" y2="8.89" width="0.1524" layer="1"/>
+<wire x1="26.67" y1="8.89" x2="26.67" y2="12.7" width="0.1524" layer="1"/>
+<wire x1="26.67" y1="12.7" x2="27.94" y2="13.97" width="0.1524" layer="1"/>
+<wire x1="27.94" y1="13.97" x2="29.21" y2="13.97" width="0.1524" layer="1"/>
 </signal>
 <signal name="3.3V">
@@
 <contactref element="LFO2" pad="K"/>
 <contactref element="LFO1" pad="K"/>
-<contactref element="STATUS" pad="A"/>
 <wire x1="35.56" y1="39.37" x2="35.179" y2="38.989" width="0.1524" layer="1"/>
 <wire x1="34.29" y1="34.29" x2="35.179" y2="35.179" width="0.1524" layer="1"/>
@@
 <wire x1="29.21" y1="1.27" x2="22.86" y2="1.27" width="0.1524" layer="1"/>
 <wire x1="22.86" y1="1.27" x2="13.97" y2="1.27" width="0.1524" layer="1"/>
-<wire x1="22.86" y1="3.81" x2="22.86" y2="1.27" width="0.1524" layer="1"/>
 <wire x1="81.28" y1="30.48" x2="82.55" y2="29.21" width="0.1524" layer="1"/>
 <wire x1="82.55" y1="29.21" x2="82.55" y2="1.27" width="0.1524" layer="1"/>
