File: modules/clock/circuits/clock.brd (EAGLE design)
At the start: 70.8 x 47 mm, 32 parts, among them IC1 4056N, IC2 4056N, IC3 4056N

Commit message: PCB correction for clock
Parts:
- added C3: 0.1uF, SparkFun-Capacitors:CAP-PTH-SMALL-KIT
Connections:
- net 5V: now also C3.2, IC1.6, IC2.6, IC3.6
- net GND: now also C3.1
Routing:
- net 5V: track 88.1 -> 162.0 mm
- net GND: track 285.0 -> 294.6 mm
- net KNOB_PIN_2: track 48.6 -> 46.3 mm
Changed lines of the file:
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@@
 <attribute name="VALUE" x="51.4858" y="18.034" size="1.27" layer="27" ratio="10" rot="R90"/>
+</element>
+<element name="C3" library="SparkFun-Capacitors" library_urn="urn:adsk.eagle:library:510" package="CAP-PTH-SMALL-KIT" package3d_urn="urn:adsk.eagle:package:37428/1" value="0.1uF" x="58.42" y="3.81" smashed="yes" rot="R180">
+<attribute name="PROD_ID" value="CAP-08370" x="58.42" y="3.81" size="1.778" layer="27" rot="R180" display="off"/>
 </element>
 </elements>
@@
 <wire x1="46.99" y1="3.81" x2="46.99" y2="1.27" width="0.1524" layer="1"/>
 <wire x1="46.99" y1="3.81" x2="46.99" y2="8.89" width="0.1524" layer="1"/>
-<wire x1="46.99" y1="1.27" x2="54.61" y2="1.27" width="0.1524" layer="1"/>
-<wire x1="54.61" y1="1.27" x2="54.61" y2="5.08" width="0.1524" layer="1"/>
-<wire x1="54.61" y1="5.08" x2="66.04" y2="5.08" width="0.1524" layer="1"/>
-<wire x1="66.04" y1="5.08" x2="68.58" y2="7.62" width="0.1524" layer="1"/>
+<wire x1="46.99" y1="1.27" x2="62.23" y2="1.27" width="0.1524" layer="1"/>
+<wire x1="62.23" y1="1.27" x2="68.58" y2="7.62" width="0.1524" layer="1"/>
 <wire x1="68.58" y1="7.62" x2="68.58" y2="19.05" width="0.1524" layer="1"/>
 </signal>
@@
 <wire x1="46.3423625" y1="33.02" x2="47.8917625" y2="34.5694" width="0.1524" layer="1"/>
 <wire x1="63.8682375" y1="34.5694" x2="65.4176375" y2="33.02" width="0.1524" layer="1"/>
-<wire x1="47.8917625" y1="34.5694" x2="63.8682375" y2="34.5694" width="0.1524" layer="1"/>
+<wire x1="47.8917625" y1="34.5694" x2="57.15" y2="34.5694" width="0.1524" layer="1"/>
+<wire x1="57.15" y1="34.5694" x2="63.8682375" y2="34.5694" width="0.1524" layer="1"/>
 <wire x1="58.42" y1="27.94" x2="59.69" y2="27.94" width="0.1524" layer="16"/>
 <wire x1="59.69" y1="27.94" x2="59.69" y2="13.7672375" width="0.1524" layer="16"/>
@@
 <wire x1="57.15" y1="13.7672375" x2="55.88" y2="12.4972375" width="0.1524" layer="16"/>
 <wire x1="55.88" y1="12.4972375" x2="55.88" y2="10.16" width="0.1524" layer="16"/>
+<contactref element="C3" pad="2"/>
+<contactref element="IC1" pad="6"/>
+<contactref element="IC2" pad="6"/>
+<contactref element="IC3" pad="6"/>
+<wire x1="53.34" y1="40.64" x2="53.34" y2="41.91" width="0.1524" layer="1"/>
+<wire x1="53.34" y1="41.91" x2="54.61" y2="43.18" width="0.1524" layer="1"/>
+<wire x1="54.61" y1="43.18" x2="57.15" y2="43.18" width="0.1524" layer="1"/>
+<wire x1="57.15" y1="43.18" x2="57.15" y2="34.5694" width="0.1524" layer="1"/>
+<wire x1="30.48" y1="40.64" x2="26.67" y2="36.83" width="0.1524" layer="1"/>
+<wire x1="26.67" y1="36.83" x2="12.7" y2="36.83" width="0.1524" layer="1"/>
+<wire x1="11.049" y1="42.9386375" x2="10.16" y2="43.8276375" width="0.1524" layer="1"/>
+<wire x1="12.7" y1="36.83" x2="11.049" y2="38.481" width="0.1524" layer="1"/>
+<wire x1="11.049" y1="38.481" x2="11.049" y2="42.9386375" width="0.1524" layer="1"/>
+<wire x1="10.16" y1="43.8276375" x2="7.62" y2="41.2876375" width="0.1524" layer="1"/>
+<wire x1="7.62" y1="40.64" x2="7.62" y2="41.2876375" width="0.1524" layer="1"/>
+<wire x1="17.78" y1="30.48" x2="8.89" y2="30.48" width="0.1524" layer="16"/>
+<wire x1="17.78" y1="30.48" x2="20.32" y2="33.02" width="0.1524" layer="16"/>
+<wire x1="57.023" y1="3.81" x2="52.07" y2="3.81" width="0.1524" layer="16"/>
+<wire x1="8.89" y1="39.37" x2="7.62" y2="40.64" width="0.1524" layer="16"/>
+<wire x1="8.89" y1="30.48" x2="8.89" y2="39.37" width="0.1524" layer="16"/>
 </signal>
 <signal name="GND">
 <contactref element="JP2" pad="6"/>
 <contactref element="FTDI" pad="1"/>
-<contactref element="ATTINY44" pad="14"/>
 <contactref element="IC1" pad="8"/>
 <contactref element="IC2" pad="8"/>
@@
 <wire x1="25.4" y1="40.64" x2="27.94" y2="40.64" width="0.1524" layer="1"/>
 <wire x1="48.26" y1="40.64" x2="50.8" y2="40.64" width="0.1524" layer="1"/>
-<wire x1="5.08" y1="40.64" x2="7.62" y2="43.18" width="0.1524" layer="1"/>
+<wire x1="5.08" y1="40.64" x2="8.89" y2="44.45" width="0.1524" layer="1"/>
 <wire x1="50.8" y1="41.91" x2="50.8" y2="40.64" width="0.1524" layer="1"/>
-<wire x1="7.62" y1="43.18" x2="13.97" y2="43.18" width="0.1524" layer="1"/>
-<wire x1="13.97" y1="43.18" x2="13.97" y2="36.83" width="0.1524" layer="1"/>
-<wire x1="13.97" y1="36.83" x2="24.13" y2="36.83" width="0.1524" layer="1"/>
-<wire x1="25.4" y1="38.1" x2="24.13" y2="36.83" width="0.1524" layer="1"/>
+<wire x1="8.89" y1="44.45" x2="13.97" y2="44.45" width="0.1524" layer="1"/>
+<wire x1="13.97" y1="44.45" x2="13.97" y2="38.1" width="0.1524" layer="1"/>
+<wire x1="13.97" y1="38.1" x2="25.4" y2="38.1" width="0.1524" layer="1"/>
 <wire x1="25.4" y1="38.1" x2="25.4" y2="40.64" width="0.1524" layer="1"/>
 <wire x1="27.94" y1="40.64" x2="27.94" y2="41.91" width="0.1524" layer="1"/>
@@
 <wire x1="29.21" y1="43.18" x2="39.37" y2="43.18" width="0.1524" layer="1"/>
 <wire x1="39.37" y1="43.18" x2="39.37" y2="38.1" width="0.1524" layer="1"/>
-<wire x1="2.54" y1="40.64" x2="8.6106" y2="34.5694" width="0.1524" layer="16"/>
-<wire x1="8.6106" y1="34.5694" x2="39.37" y2="34.5694" width="0.1524" layer="16"/>
-<wire x1="39.37" y1="34.5694" x2="39.37" y2="8.89" width="0.1524" layer="16"/>
+<wire x1="39.37" y1="20.5994" x2="39.37" y2="8.89" width="0.1524" layer="16"/>
 <wire x1="39.37" y1="38.1" x2="41.91" y2="38.1" width="0.1524" layer="1"/>
 <wire x1="41.91" y1="38.1" x2="41.91" y2="43.18" width="0.1524" layer="1"/>
@@
 <wire x1="5.08" y1="2.54" x2="6.35" y2="1.27" width="0.1524" layer="16"/>
 <wire x1="6.35" y1="1.27" x2="19.05" y2="1.27" width="0.1524" layer="16"/>
+<wire x1="68.58" y1="25.4" x2="68.58" y2="7.62" width="0.1524" layer="16"/>
+<wire x1="68.58" y1="7.62" x2="64.77" y2="3.81" width="0.1524" layer="16"/>
+<wire x1="64.77" y1="3.81" x2="62.23" y2="1.27" width="0.1524" layer="16"/>
+<wire x1="62.23" y1="1.27" x2="36.83" y2="1.27" width="0.1524" layer="16"/>
+<contactref element="ATTINY44" pad="14"/>
+<contactref element="C3" pad="1"/>
 <wire x1="66.04" y1="27.94" x2="68.58" y2="25.4" width="0.1524" layer="16"/>
-<wire x1="68.58" y1="25.4" x2="68.58" y2="7.62" width="0.1524" layer="16"/>
-<wire x1="68.58" y1="7.62" x2="66.04" y2="5.08" width="0.1524" layer="16"/>
-<wire x1="66.04" y1="5.08" x2="57.15" y2="5.08" width="0.1524" layer="16"/>
-<wire x1="57.15" y1="5.08" x2="54.61" y2="2.54" width="0.1524" layer="16"/>
-<wire x1="54.61" y1="2.54" x2="54.61" y2="1.27" width="0.1524" layer="16"/>
-<wire x1="54.61" y1="1.27" x2="36.83" y2="1.27" width="0.1524" layer="16"/>
+<wire x1="59.817" y1="3.81" x2="64.77" y2="3.81" width="0.1524" layer="16"/>
+<wire x1="2.54" y1="40.64" x2="2.54" y2="35.56" width="0.1524" layer="16"/>
+<wire x1="2.54" y1="35.56" x2="1.27" y2="34.29" width="0.1524" layer="16"/>
+<wire x1="1.27" y1="34.29" x2="1.27" y2="20.5994" width="0.1524" layer="16"/>
+<wire x1="1.27" y1="20.5994" x2="39.37" y2="20.5994" width="0.1524" layer="16"/>
 </signal>
 <signal name="RESET">

Commit message: midi2cv
Connections:
- net 5V: now also D1.3, D1.8, D2.3, D2.8, D3.3, D3.8
- net GND: no longer D1.3, D1.8, D2.3, D2.8, D3.3, D3.8
Routing:
- net 5V: track 162.0 -> 258.6 mm, vias 0 -> 1
- net GND: track 294.6 -> 215.0 mm
Changed lines of the file:
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@@
 <?xml version="1.0" encoding="utf-8"?>
 <!DOCTYPE eagle SYSTEM "eagle.dtd">
-<eagle version="9.5.2">
+<eagle version="9.6.2">
 <drawing>
 <settings>
@@
 <wire x1="8.89" y1="39.37" x2="7.62" y2="40.64" width="0.1524" layer="16"/>
 <wire x1="8.89" y1="30.48" x2="8.89" y2="39.37" width="0.1524" layer="16"/>
+<contactref element="D2" pad="3"/>
+<contactref element="D2" pad="8"/>
+<contactref element="D3" pad="3"/>
+<contactref element="D3" pad="8"/>
+<contactref element="D1" pad="3"/>
+<contactref element="D1" pad="8"/>
+<wire x1="34.24" y1="7.62" x2="29.21" y2="7.62" width="0.1524" layer="16"/>
+<wire x1="29.21" y1="7.62" x2="26.72" y2="7.62" width="0.1524" layer="16"/>
+<wire x1="22.81" y1="7.2248125" x2="22.81" y2="7.62" width="0.1524" layer="16"/>
+<wire x1="3.86" y1="7.62" x2="7.62" y2="7.62" width="0.1524" layer="16"/>
+<wire x1="7.62" y1="7.62" x2="11.38" y2="7.62" width="0.1524" layer="16"/>
+<wire x1="15.29" y1="7.62" x2="19.05" y2="7.62" width="0.1524" layer="16"/>
+<wire x1="19.05" y1="7.62" x2="22.81" y2="7.62" width="0.1524" layer="16"/>
+<wire x1="29.21" y1="7.62" x2="29.21" y2="2.3622" width="0.1524" layer="16"/>
+<wire x1="29.21" y1="2.3622" x2="27.94" y2="1.0922" width="0.1524" layer="16"/>
+<wire x1="19.05" y1="1.0922" x2="27.94" y2="1.0922" width="0.1524" layer="16"/>
+<wire x1="19.05" y1="1.0922" x2="9.0678" y2="1.0922" width="0.1524" layer="16"/>
+<wire x1="7.62" y1="2.54" x2="7.62" y2="7.62" width="0.1524" layer="16"/>
+<wire x1="9.0678" y1="1.0922" x2="7.62" y2="2.54" width="0.1524" layer="16"/>
+<wire x1="19.05" y1="7.62" x2="19.05" y2="1.0922" width="0.1524" layer="16"/>
+<wire x1="7.62" y1="7.62" x2="7.62" y2="12.7" width="0.1524" layer="16"/>
+<wire x1="7.62" y1="12.7" x2="6.35" y2="13.97" width="0.1524" layer="16"/>
+<wire x1="6.35" y1="13.97" x2="6.35" y2="19.05" width="0.1524" layer="16"/>
+<via x="6.35" y="19.05" extent="1-16" drill="0.35"/>
+<wire x1="6.35" y1="39.37" x2="7.62" y2="40.64" width="0.1524" layer="1"/>
+<wire x1="6.35" y1="19.05" x2="6.35" y2="39.37" width="0.1524" layer="1"/>
 </signal>
 <signal name="GND">
@@
 <contactref element="IC1" pad="7"/>
 <contactref element="IC2" pad="7"/>
-<contactref element="D2" pad="3"/>
-<contactref element="D2" pad="8"/>
-<contactref element="D3" pad="3"/>
-<contactref element="D3" pad="8"/>
-<contactref element="D1" pad="3"/>
-<contactref element="D1" pad="8"/>
-<wire x1="11.38" y1="7.62" x2="5.08" y2="7.62" width="0.1524" layer="16"/>
-<wire x1="5.08" y1="7.62" x2="3.86" y2="7.62" width="0.1524" layer="16"/>
-<wire x1="22.81" y1="7.62" x2="19.05" y2="7.62" width="0.1524" layer="16"/>
-<wire x1="19.05" y1="7.62" x2="15.29" y2="7.62" width="0.1524" layer="16"/>
-<wire x1="34.24" y1="7.62" x2="26.72" y2="7.62" width="0.1524" layer="16"/>
 <wire x1="2.54" y1="40.64" x2="5.08" y2="40.64" width="0.1524" layer="1"/>
 <wire x1="25.4" y1="40.64" x2="27.94" y2="40.64" width="0.1524" layer="1"/>
@@
 <wire x1="41.91" y1="43.18" x2="49.53" y2="43.18" width="0.1524" layer="1"/>
 <wire x1="49.53" y1="43.18" x2="50.8" y2="41.91" width="0.1524" layer="1"/>
-<wire x1="5.08" y1="7.62" x2="5.08" y2="2.54" width="0.1524" layer="16"/>
-<wire x1="19.05" y1="1.27" x2="36.83" y2="1.27" width="0.1524" layer="16"/>
-<wire x1="36.83" y1="1.27" x2="39.37" y2="3.81" width="0.1524" layer="16"/>
-<wire x1="22.81" y1="7.2248125" x2="22.81" y2="7.62" width="0.1524" layer="16"/>
-<wire x1="19.05" y1="7.62" x2="19.05" y2="1.27" width="0.1524" layer="16"/>
+<wire x1="39.37" y1="1.27" x2="39.37" y2="3.81" width="0.1524" layer="16"/>
 <wire x1="39.37" y1="8.89" x2="39.37" y2="3.81" width="0.1524" layer="1"/>
-<wire x1="34.24" y1="7.62" x2="35.51" y2="8.89" width="0.1524" layer="1"/>
 <wire x1="35.51" y1="8.89" x2="39.37" y2="8.89" width="0.1524" layer="1"/>
-<wire x1="3.86" y1="7.62" x2="11.38" y2="7.62" width="0.1524" layer="16"/>
-<wire x1="5.08" y1="2.54" x2="6.35" y2="1.27" width="0.1524" layer="16"/>
-<wire x1="6.35" y1="1.27" x2="19.05" y2="1.27" width="0.1524" layer="16"/>
 <wire x1="68.58" y1="25.4" x2="68.58" y2="7.62" width="0.1524" layer="16"/>
 <wire x1="68.58" y1="7.62" x2="64.77" y2="3.81" width="0.1524" layer="16"/>
 <wire x1="64.77" y1="3.81" x2="62.23" y2="1.27" width="0.1524" layer="16"/>
-<wire x1="62.23" y1="1.27" x2="36.83" y2="1.27" width="0.1524" layer="16"/>
+<wire x1="62.23" y1="1.27" x2="39.37" y2="1.27" width="0.1524" layer="16"/>
 <contactref element="ATTINY44" pad="14"/>
 <contactref element="C3" pad="1"/>

Commit message: flanger
Other:
- board text added: "+5"
- board text added: "0.1uF"
- board text added: "clk"
- board text added: "clk*8"
- board text added: "g"
Changed lines of the file:
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@@
 <hole x="68.58" y="44.45" drill="3.200146875"/>
 <hole x="67.31" y="2.54" drill="3.200146875"/>
+<text x="60.96" y="6.35" size="0.8128" layer="21">0.1uF</text>
+<text x="57.15" y="1.27" size="0.8128" layer="21">0.1uF</text>
+<text x="39.37" y="1.27" size="0.8128" layer="21" rot="R180">g</text>
+<text x="36.83" y="7.62" size="0.8128" layer="21">g</text>
+<text x="53.34" y="1.27" size="0.8128" layer="21" rot="R180">+5</text>
+<text x="45.72" y="1.27" size="0.8128" layer="21" rot="R180">clk</text>
+<text x="43.18" y="1.27" size="0.8128" layer="21" rot="R180">clk*8</text>
 </plain>
 <attributes>
@@
 </element>
 <element name="FTDI" library="pinhead" library_urn="urn:adsk.eagle:library:325" package="1X06" package3d_urn="urn:adsk.eagle:package:22472/2" value="" x="45.72" y="8.89" smashed="yes">
-<attribute name="NAME" x="38.0238" y="10.7188" size="1.27" layer="25" ratio="10"/>
+<attribute name="NAME" x="38.0238" y="10.7188" size="1.27" layer="21" ratio="10"/>
 <attribute name="POPULARITY" value="79" x="67.31" y="-35.56" size="1.778" layer="27" display="off"/>
 <attribute name="VALUE" x="38.1" y="5.715" size="1.27" layer="27"/>
@@
 <attribute name="NAME" x="21.971" y="39.751" size="1.27" layer="25" ratio="10" rot="R270"/>
 <attribute name="POPULARITY" value="0" x="-34.29" y="62.23" size="1.778" layer="27" rot="R180" display="off"/>
-<attribute name="VALUE" x="18.923" y="37.465" size="1.27" layer="27" ratio="10" rot="R180"/>
+<attribute name="VALUE" x="18.923" y="37.465" size="1.27" layer="21" ratio="10" rot="R180"/>
 </element>
 <element name="IC2" library="40xx" library_urn="urn:adsk.eagle:library:80" package="DIL16" package3d_urn="urn:adsk.eagle:package:922/2" value="4056N" x="57.15" y="36.83" smashed="yes" rot="R180">
 <attribute name="POPULARITY" value="0" x="33.02" y="73.66" size="1.778" layer="27" rot="R180" display="off"/>
-<attribute name="VALUE" x="64.643" y="37.465" size="1.27" layer="27" ratio="10" rot="R180"/>
+<attribute name="VALUE" x="64.643" y="37.465" size="1.27" layer="21" ratio="10" rot="R180"/>
 </element>
 <element name="IC3" library="40xx" library_urn="urn:adsk.eagle:library:80" package="DIL16" package3d_urn="urn:adsk.eagle:package:922/2" value="4056N" x="34.29" y="36.83" smashed="yes" rot="R180">
 <attribute name="NAME" x="44.831" y="39.751" size="1.27" layer="25" ratio="10" rot="R270"/>
 <attribute name="POPULARITY" value="0" x="-12.7" y="73.66" size="1.778" layer="27" rot="R180" display="off"/>
-<attribute name="VALUE" x="41.783" y="37.465" size="1.27" layer="27" ratio="10" rot="R180"/>
+<attribute name="VALUE" x="41.783" y="37.465" size="1.27" layer="21" ratio="10" rot="R180"/>
 </element>
 <element name="JP2" library="pinhead" library_urn="urn:adsk.eagle:library:325" package="1X06" package3d_urn="urn:adsk.eagle:package:22472/2" value="" x="45.72" y="3.81" smashed="yes" rot="R180">
-<attribute name="NAME" x="53.4162" y="1.9812" size="1.27" layer="25" ratio="10" rot="R180"/>
 <attribute name="POPULARITY" value="79" x="7.62" y="48.26" size="1.778" layer="27" rot="R180" display="off"/>
 <attribute name="VALUE" x="53.34" y="6.985" size="1.27" layer="27" rot="R180"/>
@@
 <element name="R1" library="adafruit" library_urn="urn:adsk.eagle:library:420" package="0207/12" package3d_urn="urn:adsk.eagle:package:6240598/1" value="10k" x="55.88" y="16.51" smashed="yes" rot="R270">
 <attribute name="NAME" x="57.277" y="19.685" size="1.27" layer="25" ratio="10" rot="R270"/>
-<attribute name="VALUE" x="55.1942" y="18.796" size="1.27" layer="27" ratio="10" rot="R270"/>
+<attribute name="VALUE" x="55.1942" y="18.796" size="1.27" layer="21" ratio="10" rot="R270"/>
 </element>
 <element name="R10" library="adafruit" library_urn="urn:adsk.eagle:library:420" package="0207/12" package3d_urn="urn:adsk.eagle:package:6240598/1" value="150" x="20.32" y="22.86" smashed="yes" rot="R90">
@@
 </element>
 <element name="R18" library="adafruit" library_urn="urn:adsk.eagle:library:420" package="0207/12" package3d_urn="urn:adsk.eagle:package:6240598/1" value="150" x="2.54" y="22.86" smashed="yes" rot="R90">
-<attribute name="VALUE" x="3.2258" y="20.574" size="1.27" layer="27" ratio="10" rot="R90"/>
+<attribute name="VALUE" x="3.2258" y="20.574" size="1.27" layer="21" ratio="10" rot="R90"/>
 </element>
 <element name="R19" library="adafruit" library_urn="urn:adsk.eagle:library:420" package="0207/12" package3d_urn="urn:adsk.eagle:package:6240598/1" value="150" x="5.08" y="22.86" smashed="yes" rot="R90">
