File: modules/flanger/circuit/flanger.sch (EAGLE design)
At the start: 28 parts, among them IC1 LM324N, U1 ATTINY84

Commit message: flanger
Parts:
- removed JP1: (no value), pinhead:PINHD-1X4
- removed R12: 100K, rcl:R-EU_0207/10
- added C5: 0.01uF, capacitor-wima:C5/2.5
- added C6, C7: 0.1uF, capacitor-wima:C5/2.5
- added FTDI, KNOBS, POWER: (no value), adafruit:PINHD-1X6
- added R18: 10K, rcl:R-EU_0207/10
- added VR2: 100k, SparkFun-Resistors:TRIMPOT-PTH-10MM-KNOB-1/2W-10%
- C3, C4: device capacitor-wima:C7.5/3 -> capacitor-wima:C5/2.5
- R15: value 100K -> 220K
- U1: value ATTINY84 -> ATTINY84ATTINY84-20PU; device SparkFun-IC-Microcontroller:ATTINY84 -> SparkFun-IC-Microcontroller:ATTINY84ATTINY84-20PU
Connections:
- new net DEPTH: KNOBS.5, U1.(SCL/SCK/ADC4)PA4
- new net MANUAL: KNOBS.4, U1.(ADC0)PA0
- new net N$14: C5.2, R16.1
- new net N$16: C7.1, R18.1, U1.(!RESET!)PB3
- new net RATE: KNOBS.6, U1.(ADC3)PA3
- new net RESET: C7.2, FTDI.6
- new net RX: FTDI.5, U1.(ADC1)PA1
- new net SPARE1: KNOBS.1, U1.(INT0)PB2
- new net SPARE2: KNOBS.2, U1.(XTAL2)PB1
- new net SPARE3: KNOBS.3, U1.(ADC7)PA7
- new net TX: FTDI.4, U1.(ADC2)PA2
- net +12V: now also POWER.2
- net +5V: now also C6.2, POWER.1, R18.2, U1.VCC
- net -12V: now also POWER.3
- net CLK1: now also U1.(RX/POCI/ADC5)PA5; no longer U1.(ADC7)PA7
- net GND: now also C6.1, FTDI.1, POWER.6, U1.GND
- net N$11: now also VR2.WIPER; no longer R12.2
- net N$15: now also C5.1; no longer R16.1
- net N$7: now also VR2.CCW; no longer R12.1
- net SIGNAL_IN: now also POWER.4
- net SIGNAL_OUT: now also POWER.5
Other:
- note added: "Connections"
- note added: "Oscillator"
- moved on the sheet: FEEDBACK_POT10K1, U1, V3208D
