File: modules/vcf/circuit/vcf.brd (EAGLE design)
At the start: 100 x 80 mm, 18 parts, among them IC1 CEM3320

Commit message: vcf done
Parts:
- added C6: 1uF, rcl:C025-030X050
- added IC2: LM324N, linear:DIL14
- added JP1, JP2: (no value), pinhead:1X04
- added NOISE: (no value), adafruit:1X01
- added R13: 16.5K, adafruit:0204/7
- added R14: 500, adafruit:0204/7
- added R15: 100K, adafruit:0204/7
- added R16: 3.6K, adafruit:0204/7
- added R17, R18: 50K, adafruit:0204/7
- moved R12 159.7 mm to (34.3, 50.8), turned to 180 degrees
- moved R9 148.8 mm to (34.3, 53.3), turned to 180 degrees
- moved R8 146.6 mm to (34.3, 55.9)
- moved C5 145.3 mm to (29.2, 30.5)
- moved R11 144.3 mm to (43.2, 31.8)
- moved R10 143.9 mm to (14.0, 53.3), turned to 180 degrees
- moved R7 137.0 mm to (24.1, 55.9)
- moved R6 127.8 mm to (14.0, 55.9)
- moved R5 123.0 mm to (43.2, 34.3)
- moved R4 109.0 mm to (27.9, 34.3)
- moved R3 98.6 mm to (17.8, 34.3)
- moved C4 94.8 mm to (5.08, 43.2), turned to 180 degrees
- moved C1 91.6 mm to (5.08, 54.6), turned to 180 degrees
- moved C3 91.6 mm to (5.08, 47.0), turned to 180 degrees
- moved C2 82.3 mm to (5.08, 50.8), turned to 180 degrees
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Connections:
- new net +5V: JP1.3, R13.1
- new net CV_F_IN: JP2.1, R15.1
- new net CV_RES: IC2.6, IC2.7, R18.1
- new net CV_RES_IN: IC2.5, JP2.2
- new net N$13: IC2.3, R13.2, R14.2
- new net N$15: IC2.2, NOISE.1, R15.2, R16.1
- new net N$16: C6.2, R2.1
- new net N$17: IC1.8, R17.2
- new net N$18: IC1.9, R18.2
- new net N$20: C5.2, IC2.10
- net +12V: now also IC2.4, JP1.1
- net -12V: now also IC2.11, JP1.2
- net CV_F: now also IC2.1, R16.2
- net GND: now also JP1.4, R14.1
- net IN: now also C6.1, JP2.3; no longer R2.1
- net OUT: now also IC2.8, IC2.9, JP2.4, R17.1; no longer C5.2
Routing:
- net -12V: track 0.00 -> 91.0 mm, vias 0 -> 1
- net GND: track 0.00 -> 69.7 mm
- net N$15: track 0.00 -> 65.9 mm
- net N$9: track 0.00 -> 63.6 mm
- net CV_RES_IN: track 0.00 -> 56.6 mm, vias 0 -> 1
- net OUT: track 0.00 -> 49.8 mm
- net N$20: track 0.00 -> 46.6 mm
- net CV_F: track 0.00 -> 44.3 mm
- net +12V: track 0.00 -> 39.2 mm
- net N$12: track 0.00 -> 39.2 mm
- net N$4: track 0.00 -> 38.0 mm
- net CV_F_IN: track 0.00 -> 37.7 mm
- net N$8: track 0.00 -> 33.0 mm
- net N$14: track 0.00 -> 27.1 mm, vias 0 -> 1
- net +5V: track 0.00 -> 23.4 mm
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Other:
- board size 100 x 80 mm -> 60.6 x 34.3 mm
- board text added: "+12"
- board text added: "-12"
- board text added: "4 STAGE LOW PASS FILTER"
- board text added: "5"
- board text added: "CUT"
- board text added: "DUMAIS"
- board text added: "G"
- board text added: "IN"
- board text added: "OUT"
- board text added: "RES"

Commit message: a few misc changes
Connections:
- removed net N$20: C5.2, IC2.10
- new net RES_FDB: C5.2, IC2.10, R17.1
- net OUT: no longer R17.1
Routing:
- net RES_FDB: track 0.00 -> 52.2 mm
- net N$20: track 46.6 -> 0.00 mm
- net CV_F_IN: track 37.7 -> 38.7 mm
- net OUT: vias 0 -> 1
Changed lines of the file:
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@@
 <signal name="OUT">
 <contactref element="JP2" pad="4"/>
-<contactref element="R17" pad="1"/>
 <contactref element="IC2" pad="8"/>
 <contactref element="IC2" pad="9"/>
 <wire x1="52.07" y1="43.18" x2="52.07" y2="40.64" width="0.1524" layer="16"/>
-<wire x1="34.29" y1="27.94" x2="35.56" y2="26.67" width="0.1524" layer="16"/>
-<wire x1="35.56" y1="26.67" x2="50.8" y2="26.67" width="0.1524" layer="16"/>
-<wire x1="50.8" y1="26.67" x2="52.07" y2="27.94" width="0.1524" layer="16"/>
+<wire x1="52.07" y1="27.94" x2="50.8" y2="26.67" width="0.1524" layer="16"/>
 <wire x1="52.07" y1="27.94" x2="52.07" y2="40.64" width="0.1524" layer="16"/>
 <wire x1="19.05" y1="29.21" x2="27.94" y2="29.21" width="0.1524" layer="1"/>
-<wire x1="27.94" y1="29.21" x2="29.21" y2="27.94" width="0.1524" layer="1"/>
-<wire x1="29.21" y1="27.94" x2="34.29" y2="27.94" width="0.1524" layer="1"/>
+<wire x1="50.8" y1="26.67" x2="31.75" y2="26.67" width="0.1524" layer="16"/>
+<via x="31.75" y="26.67" extent="1-16" drill="0.35"/>
+<wire x1="30.48" y1="26.67" x2="31.75" y2="26.67" width="0.1524" layer="1"/>
+<wire x1="27.94" y1="29.21" x2="30.48" y2="26.67" width="0.1524" layer="1"/>
 </signal>
 <signal name="CV_F">
@@
 <contactref element="JP2" pad="1"/>
 <contactref element="R15" pad="1"/>
-<wire x1="46.99" y1="29.21" x2="44.45" y2="26.67" width="0.1524" layer="1"/>
-<wire x1="44.45" y1="26.67" x2="13.97" y2="26.67" width="0.1524" layer="1"/>
-<wire x1="13.97" y1="26.67" x2="11.43" y2="29.21" width="0.1524" layer="1"/>
+<wire x1="46.99" y1="29.21" x2="43.18" y2="25.4" width="0.1524" layer="1"/>
+<wire x1="43.18" y1="25.4" x2="15.24" y2="25.4" width="0.1524" layer="1"/>
+<wire x1="15.24" y1="25.4" x2="11.43" y2="29.21" width="0.1524" layer="1"/>
 </signal>
 <signal name="CV_RES_IN">
@@
 <wire x1="43.18" y1="39.37" x2="44.45" y2="40.64" width="0.1524" layer="1"/>
 </signal>
-<signal name="N$20">
+<signal name="RES_FDB">
+<contactref element="R17" pad="1"/>
 <contactref element="C5" pad="2"/>
 <contactref element="IC2" pad="10"/>
@@
 <wire x1="54.3052" y1="33.57335" x2="54.0032" y2="33.27135" width="0.1524" layer="16"/>
 <wire x1="54.0032" y1="33.27135" x2="54.0032" y2="28.6032" width="0.1524" layer="16"/>
-<wire x1="33.02" y1="25.4" x2="50.8" y2="25.4" width="0.1524" layer="16"/>
+<wire x1="31.75" y1="25.4" x2="50.8" y2="25.4" width="0.1524" layer="16"/>
 <wire x1="54.3052" y1="43.4848" x2="54.3052" y2="33.57335" width="0.1524" layer="16"/>
 <wire x1="54.0032" y1="28.6032" x2="50.8" y2="25.4" width="0.1524" layer="16"/>
-<wire x1="30.48" y1="30.48" x2="30.48" y2="27.94" width="0.1524" layer="16"/>
-<wire x1="30.48" y1="27.94" x2="33.02" y2="25.4" width="0.1524" layer="16"/>
+<wire x1="30.48" y1="30.48" x2="30.48" y2="26.67" width="0.1524" layer="16"/>
+<wire x1="30.48" y1="26.67" x2="31.75" y2="25.4" width="0.1524" layer="16"/>
+<wire x1="34.29" y1="27.94" x2="31.75" y2="30.48" width="0.1524" layer="1"/>
+<wire x1="31.75" y1="30.48" x2="30.48" y2="30.48" width="0.1524" layer="1"/>
 </signal>
 </signals>
