File: modules/vcf/circuit/vcf.sch (EAGLE design)
At the start: 18 parts, among them IC1 CEM3320

Commit message: vcf done
Parts:
- added C6: 1uF, rcl:C-EU025-030X050
- added IC2: LM324N, linear:LM324N
- added JP1, JP2: (no value), pinhead:PINHD-1X4
- added NOISE: (no value), adafruit:PINHD-1X1
- added R13: 16.5K, adafruit:R-US_0204/7
- added R14: 500, adafruit:R-US_0204/7
- added R15: 100K, adafruit:R-US_0204/7
- added R16: 3.6K, adafruit:R-US_0204/7
- added R17, R18: 50K, adafruit:R-US_0204/7
Connections:
- new net +5V: JP1.3, R13.1
- new net CV_F_IN: JP2.1, R15.1
- new net CV_RES: IC2B.-IN, IC2B.OUT, R18.1
- new net CV_RES_IN: IC2B.+IN, JP2.2
- new net N$13: IC2A.+IN, R13.2, R14.2
- new net N$15: IC2A.-IN, NOISE.1, R15.2, R16.1
- new net N$16: C6.2, R2.1
- new net N$17: IC1.8, R17.2
- new net N$18: IC1.9, R18.2
- new net N$20: C5.2, IC2C.+IN
- net +12V: now also IC2P.V+, JP1.1
- net -12V: now also IC2P.V-, JP1.2
- net CV_F: now also IC2A.OUT, R16.2
- net GND: now also JP1.4, R14.1
- net IN: now also C6.1, JP2.3; no longer R2.1
- net OUT: now also IC2C.-IN, IC2C.OUT, JP2.4, R17.1; no longer C5.2
Other:
- note added: "0V -> 151mV 5V -> -28mV"
- note added: "CV inputs are 0V .. 5V IN and OUT are -5V .. +5V"

Commit message: a few misc changes
Connections:
- removed net N$20: C5.2, IC2C.+IN
- new net RES_FDB: C5.2, IC2C.+IN, R17.1
- net OUT: no longer R17.1
Changed lines of the file:
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@@
 </instance>
 <instance part="R17" gate="G$1" x="17.78" y="33.02" smashed="yes">
-<attribute name="VALUE" x="11.43" y="34.798" size="1.778" layer="96"/>
+<attribute name="VALUE" x="13.97" y="34.798" size="1.778" layer="96"/>
 </instance>
 <instance part="R18" gate="G$1" x="17.78" y="30.48" smashed="yes">
@@
 </segment>
 <segment>
-<pinref part="R17" gate="G$1" pin="1"/>
-<wire x1="12.7" y1="33.02" x2="7.62" y2="33.02" width="0.1524" layer="91"/>
-<wire x1="7.62" y1="33.02" x2="7.62" y2="35.56" width="0.1524" layer="91"/>
-<wire x1="7.62" y1="35.56" x2="0" y2="35.56" width="0.1524" layer="91"/>
-<label x="0" y="35.56" size="1.778" layer="95" rot="R180" xref="yes"/>
-</segment>
-<segment>
 <pinref part="IC2" gate="C" pin="OUT"/>
 <wire x1="137.16" y1="66.04" x2="149.86" y2="66.04" width="0.1524" layer="91"/>
@@
 <segment>
 <pinref part="R18" gate="G$1" pin="1"/>
-<wire x1="12.7" y1="30.48" x2="10.16" y2="30.48" width="0.1524" layer="91"/>
-<wire x1="10.16" y1="30.48" x2="10.16" y2="25.4" width="0.1524" layer="91"/>
-<wire x1="10.16" y1="25.4" x2="7.62" y2="25.4" width="0.1524" layer="91"/>
-<label x="7.62" y="25.4" size="1.778" layer="95" rot="R180" xref="yes"/>
-</segment>
-</net>
-<net name="N$20" class="0">
+<wire x1="12.7" y1="30.48" x2="7.62" y2="30.48" width="0.1524" layer="91"/>
+<label x="7.62" y="30.48" size="1.778" layer="95" rot="R180" xref="yes"/>
+</segment>
+</net>
+<net name="RES_FDB" class="0">
+<segment>
+<pinref part="R17" gate="G$1" pin="1"/>
+<wire x1="12.7" y1="33.02" x2="10.16" y2="33.02" width="0.1524" layer="91"/>
+<wire x1="10.16" y1="33.02" x2="10.16" y2="35.56" width="0.1524" layer="91"/>
+<wire x1="10.16" y1="35.56" x2="7.62" y2="35.56" width="0.1524" layer="91"/>
+<label x="7.62" y="35.56" size="1.778" layer="95" rot="R180" xref="yes"/>
+</segment>
 <segment>
 <pinref part="C5" gate="G$1" pin="2"/>
 <pinref part="IC2" gate="C" pin="+IN"/>
-<wire x1="104.14" y1="68.58" x2="121.92" y2="68.58" width="0.1524" layer="91"/>
-</segment>
-</net>
+<wire x1="104.14" y1="68.58" x2="109.22" y2="68.58" width="0.1524" layer="91"/>
+<wire x1="109.22" y1="68.58" x2="121.92" y2="68.58" width="0.1524" layer="91"/>
+<wire x1="109.22" y1="68.58" x2="109.22" y2="48.26" width="0.1524" layer="91"/>
+<junction x="109.22" y="68.58"/>
+<label x="109.22" y="48.26" size="1.778" layer="95" rot="R270" xref="yes"/>
+</segment>
+</net>
