File: modules/drum/circuit/drums.brd (EAGLE design)
At the start: 100 x 80 mm, 80 parts, among them IC1 LM324N, IC2 LM324N, Q1 2N3904, Q2 2N3904

Commit message: Drums
Parts:
- removed METAL_POT: metal_pot, pinhead:1X03
- added 1M1, 1M2: 220, SparkFun-Resistors:AXIAL-0.3
- added C18, C19, C20: 100nF, capacitor-wima:C5B3
- added D6: 1A/50V/1.1V, SparkFun-DiscreteSemi:DIODE-1N4001-KIT
- added OK1: 6N138, optocoupler:DIL08
- added R38, R39, R41, R42, R43, R44, R45: 100k, SparkFun-Resistors:AXIAL-0.3
- added R40: 10k, SparkFun-Resistors:AXIAL-0.3
- R11: value 100k -> 100
- R12, R23: value 1k -> 100k
- R19: value 100K -> 100k
- R2: value 1k -> 10k
- R20: value 50K -> 100k
- R21: value 100K -> 100
- R22: value 100k -> 10k
- moved R20 232.8 mm to (-76.2, -158.8)
- moved R19 230.5 mm to (-76.2, -154.9)
- moved R12 224.9 mm to (-76.2, -151.1)
- moved R11 223.7 mm to (-76.2, -147.3)
- moved R23 193.2 mm to (-76.2, -108.0)
- moved D2 193.0 mm to (-74.9, -138.4)
- moved R22 176.7 mm to (-76.2, -104.1)
- moved D3 152.7 mm to (-74.9, -99.1)
- moved R1 109.2 mm to (-76.2, -44.5)
Connections:
- removed net N$1: METAL_POT.2, NOISE_CHIP.8
- removed net N$13: IC2.3, R11.P$2, R12.P$2
- removed net N$14: C7.2, IC2.1, R13.P$2, R15.P$2, R20.P$1
- removed net N$21: IC2.6, R19.P$1, R20.P$2
- removed net N$8: D2.A, SNARE_TRIGGER.2
- new net BD_TRIGGER: NOISE_CHIP.2, R12.P$2
- new net DIN5_4: 1M2.P$2
- new net DIN5_5: D2.A, OK1.3
- new net HH_TRIGGER: NOISE_CHIP.5, R11.P$2
- new net MIDI_RX: 1M1.P$1, NOISE_CHIP.7, OK1.6
- new net N$15: C19.1, R19.P$1, R42.P$2, WOODBLOCK_TRIGGER.2
- new net N$28: D6.C, IC1.10, R40.P$2
- new net N$47: R41.P$2, WOODBLOCK_TRIGGER.1
- new net N$49: C19.2, D6.A, R43.P$2
- new net N$5: BD_TRIGGER.1, R38.P$2
- new net N$50: C20.2, D3.A, R45.P$2
- new net SNARE_TRIGGER: NOISE_CHIP.13, R20.P$2
- new net WB_TRIGGER: NOISE_CHIP.3, R19.P$2
- net +5V: now also 1M1.P$2, OK1.8, R23.P$1, R38.P$1, R41.P$1; no longer BD_TRIGGER.1, METAL_POT.1, SNARE_TRIGGER.1, WOODBLOCK_TRIGGER.1
- net BD_OUT: now also C7.2, IC2.1, R13.P$2, R15.P$2; no longer IC2.7, R19.P$2
- net GND: now also OK1.5, R1.P$1, R22.P$1, R39.P$1, R40.P$1, R42.P$1, R43.P$1, R44.P$1, R45.P$1; no longer IC2.5, METAL_POT.3, R12.P$1, R23.P$1
- net N$12: now also 1M2.P$1, OK1.2; no longer R11.P$1
- net N$2: now also C18.1, R12.P$1, R39.P$2; no longer D1.A
- net N$25: now also C20.1, R20.P$1, R44.P$2, SNARE_TRIGGER.2; no longer D3.A, WOODBLOCK_TRIGGER.2
- net N$26: now also IC2.3, R22.P$2; no longer R22.P$1
- net N$27: now also SNARE_TRIGGER.1; no longer IC1.10, R22.P$2
- net N$3: now also IC1.3, R2.P$2; no longer R1.P$1
- net N$32: now also R11.P$1
- net N$4: now also C18.2, D1.A; no longer IC1.3, R2.P$2
- net NOISE: now also NOISE_CHIP.8; no longer NOISE_CHIP.7

Commit message: drum board
Parts:
- added 10K_POT8, 10K_POT9, CLING_TRIGGER: (no value), pinhead:1X02
- added 1M3, 1M4, R49: 1k, SparkFun-Resistors:AXIAL-0.3
- added C21, C22, C24, C26, C28: 100nF, capacitor-wima:C5B3
- added C23: 10uF, rcl:TT5D11
- added C25, C27: 330nF, capacitor-wima:C5B3
- added D7, D8: 1A/50V/1.1V, SparkFun-DiscreteSemi:DIODE-1N4001-KIT
- added IC3: 7905, linear:TO220H
- added IC4: 7805T, adafruit:TO220H
- added Q3: 2N3904, transistor-small-signal:TO92D
- added R46: 1M, SparkFun-Resistors:AXIAL-0.3
- added R47, R48: 47K, SparkFun-Resistors:AXIAL-0.3
- added R50: 100, SparkFun-Resistors:AXIAL-0.3
- added R51: 2.2K, SparkFun-Resistors:AXIAL-0.3
- added R52, R54, R55, R56, R57: 100k, SparkFun-Resistors:AXIAL-0.3
- added R53, R59: 10k, SparkFun-Resistors:AXIAL-0.3
- added R58: 100K, SparkFun-Resistors:AXIAL-0.3
- moved R20 254.2 mm to (55.9, 58.4), turned to 270 degrees
- moved R19 225.9 mm to (54.6, 29.2)
- moved R12 212.4 mm to (38.1, 27.9)
- moved R11 211.4 mm to (38.1, 30.5)
- moved FTDI 155.2 mm to (62.2, 50.8), turned to 180 degrees
- moved C4 144.2 mm to (58.4, 31.8)
- moved R25 141.0 mm to (57.1, 35.6), turned to 180 degrees
- moved R29 134.0 mm to (55.9, 16.5)
- moved IC2 110.9 mm to (85.1, 43.2)
- moved C1 110.3 mm to (90.2, 54.6), turned to 270 degrees
- moved NOISE_CHIP 109.7 mm to (61.0, 43.2)
- moved IC1 108.1 mm to (36.8, 43.2)
- moved BD_TRIGGER 89.9 mm to (3.81, 5.08), turned to 90 degrees
- moved 10K_POT4 83.2 mm to (8.89, 6.35), turned to 90 degrees
- moved 10K_POT5 79.0 mm to (8.89, 12.7), turned to 90 degrees
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Connections:
- new net 10K_POT3: 10K_POT9.1, R47.P$1, R48.P$1
- new net BD_OUT1: C22.2, IC2.7, R46.P$2, R48.P$2, R59.P$2
- new net CLING_OUT: IC1.6, IC1.7, R58.P$1
- new net CLING_TRIGGER: NOISE_CHIP.10, R57.P$2
- new net GND2: 1M4.P$1, C27.1, IC3.2, JP1.3
- new net N$1: 10K_POT8.1, C21.2, C22.1, R49.P$2
- new net N$13: 10K_POT8.2, R49.P$1, R50.P$2
- new net N$14: 10K_POT9.2, R51.P$1
- new net N$21: C23.+, R51.P$2
- new net N$51: Q3.B, R52.P$2
- new net N$52: D8.C, Q3.C
- new net N$53: D8.A, IC1.5, R59.P$1
- new net N$54: C24.1, CLING_TRIGGER.2, R55.P$2, R57.P$1
- new net N$55: D7.C, IC2.5, R53.P$2
- new net N$56: CLING_TRIGGER.1, R54.P$2
- new net N$57: C24.2, D7.A, R56.P$2
- new net N$8: C21.1, IC2.6, R46.P$1, R47.P$2
- net +12V: now also 1M3.P$2, C25.2, IC4.1
- net +5V: now also C26.2, IC4.3, R54.P$1
- net -5V: now also C28.1, IC3.3
- net GND: now also 1M3.P$1, 1M4.P$2, C23.-, C25.1, C26.1, C27.2, C28.2, IC3.1, IC4.2, Q3.E, R50.P$1, R53.P$1, R55.P$1, R56.P$1; no longer JP1.3
- net METALIC: now also R52.P$1
- net N$34: now also R58.P$2
Routing:
- net +5V: track 0.00 -> 213.1 mm
- net -5V: track 0.00 -> 85.9 mm
- net BD_OUT1: track 0.00 -> 48.9 mm
- net N$8: track 0.00 -> 42.1 mm, vias 0 -> 1
- net CLING_TRIGGER: track 0.00 -> 34.8 mm, vias 0 -> 1
- net N$51: track 0.00 -> 21.1 mm
- net N$57: track 0.00 -> 13.8 mm
- net N$55: track 0.00 -> 10.5 mm
- net WB_TRIGGER: track 0.00 -> 10.2 mm
- net SNARE_TRIGGER: track 0.00 -> 9.72 mm
- net N$37: track 0.00 -> 7.62 mm
- net N$54: track 0.00 -> 6.35 mm
- net N$21: track 0.00 -> 6.35 mm
- net HH_OUT: track 0.00 -> 5.61 mm
- net 10K_POT3: track 0.00 -> 5.08 mm
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
Commit message: drum board cleanup
Parts:
- added JP2: (no value), adafruit:1X03
- moved R45 213.8 mm to (77.5, 33.0), turned to 90 degrees
- moved R44 211.9 mm to (74.9, 36.8), turned to 90 degrees
- moved R22 207.9 mm to (80.0, 33.0), turned to 90 degrees
- moved D3 204.7 mm to (82.5, 31.8), turned to 90 degrees
- moved C20 191.6 mm to (80.0, 22.9)
- moved R23 180.7 mm to (36.8, 33.0), turned to 270 degrees
- moved 1M1 180.0 mm to (21.6, 17.8), turned to 180 degrees
- moved 1M2 174.9 mm to (14.0, 6.35), turned to 90 degrees
- moved D2 170.8 mm to (21.6, 2.54), turned to 180 degrees
- moved R40 167.1 mm to (38.1, 53.3)
- moved D6 165.3 mm to (44.5, 50.8), turned to 180 degrees
- moved OK1 164.9 mm to (21.6, 10.2)
- moved R16 159.0 mm to (90.2, 77.5)
- moved R34 158.1 mm to (88.9, 66.0), turned to 90 degrees
- moved R43 149.4 mm to (41.9, 11.4), turned to 180 degrees
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Connections:
- net DIN5_4: now also JP2.1
- net DIN5_5: now also JP2.2
- net GND: now also JP2.3
Routing:
- net N$51: track 21.1 -> 0.64 mm
- net DIN5_4: track 0.00 -> 15.8 mm
- net DIN5_5: track 0.00 -> 15.0 mm
- net GND: track 2.54 -> 15.0 mm
- net WB_TRIGGER: track 10.2 -> 0.00 mm
- net N$12: track 0.00 -> 9.42 mm
- net MIDI_RX: track 0.00 -> 6.35 mm
- net +5V: track 213.1 -> 215.7 mm
- net N$37: track 7.62 -> 6.35 mm

Commit message: drum machine
Parts:
- removed 1M3, 1M4: 1k, SparkFun-Resistors:AXIAL-0.3
- removed C25, C27: 330nF, capacitor-wima:C5B3
- removed C26, C28: 100nF, capacitor-wima:C5B3
- removed IC3: 7905, linear:TO220H
- removed IC4: 7805T, adafruit:TO220H
- removed JP1: (no value), pinhead:1X04
- added JP3: (no value), pinhead:1X06
- added LIMIT_SWITCH, LIM_SWITCH1, LOW_BIT_NOISE: (no value), pinhead:1X02
- moved C11 126.2 mm to (94.0, 57.1), turned to 270 degrees
- moved C8 109.8 mm to (59.7, 17.8), turned to 180 degrees
- moved HH_TRIGGER 108.6 mm to (99.1, 63.5), turned to 180 degrees
- moved R55 88.2 mm to (99.1, 26.7), turned to 90 degrees
- moved 10K_POT4 86.3 mm to (81.3, 53.3), turned to 180 degrees
- moved C5 84.3 mm to (48.3, 15.2), turned to 270 degrees
- moved R29 79.1 mm to (101.6, 57.1), turned to 90 degrees
- moved R30 78.8 mm to (96.5, 43.2), turned to 90 degrees
- moved R50 74.5 mm to (102.9, 1.27), turned to 180 degrees
- moved 10K_POT8 74.0 mm to (94.0, 1.27)
- moved R49 73.8 mm to (78.7, 1.27)
- moved R17 73.3 mm to (82.5, 14.0), turned to 180 degrees
- moved 10K_POT6 68.8 mm to (58.4, 72.4), turned to 180 degrees
- moved R18 66.9 mm to (64.8, 21.6), turned to 270 degrees
- moved 10K_POT5 63.4 mm to (43.2, 66.0), turned to 0 degrees
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Connections:
- removed net -5V: C28.1, IC1.11, IC2.11, IC3.3
- removed net GND2: 1M4.P$1, C27.1, IC3.2, JP1.3
- new net -12V: IC1.11, IC2.11, JP3.2
- new net N$58: LIM_SWITCH1.2, R6.P$2
- new net N$59: LIMIT_SWITCH.2, R49.P$2
- new net N$60: LOW_BIT_NOISE.1, NOISE_CHIP.9
- net +12V: now also IC1.4, IC2.4, JP3.1; no longer 1M3.P$2, C25.2, IC4.1, JP1.1
- net +5V: now also JP3.6; no longer C26.2, IC1.4, IC2.4, IC4.3
- net GND: now also JP3.3, LOW_BIT_NOISE.2; no longer 1M3.P$1, 1M4.P$2, C25.1, C26.1, C27.2, C28.2, IC3.1, IC4.2
- net N$1: now also LIMIT_SWITCH.1; no longer R49.P$2
- net N$6: now also LIM_SWITCH1.1; no longer R6.P$2
- net OUT: now also JP3.4; no longer JP1.4
Routing:
- net GND: track 15.0 -> 444.8 mm, vias 0 -> 1
- net BD_OUT: track 0.00 -> 155.6 mm, vias 0 -> 1
- net -5V: track 85.9 -> 0.00 mm
- net N$34: track 0.00 -> 79.9 mm
- net +12V: track 0.00 -> 79.1 mm
- net -12V: track 0.00 -> 71.5 mm
- net MIDI_RX: track 6.35 -> 61.6 mm
- net N$6: track 0.00 -> 41.5 mm
- net N$25: track 0.00 -> 40.2 mm
- net N$15: track 0.00 -> 35.1 mm
- net N$17: track 0.00 -> 32.1 mm
- net N$32: track 0.00 -> 30.1 mm
- net N$33: track 0.00 -> 29.6 mm
- net N$48: track 5.08 -> 34.2 mm
- net N$36: track 0.00 -> 27.7 mm
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Other:
- board size 100 x 80 mm -> 178.7 x 113 mm

Commit message: drum machine
Parts:
- moved D8 44.6 mm to (102.9, 8.89), turned to 90 degrees
- moved R59 20.5 mm to (77.5, 5.08)
- moved D6 20.4 mm to (45.7, 30.5), turned to 90 degrees
- moved Q3 17.8 mm to (106.7, 50.8)
- moved R50 9.25 mm to (100.3, 10.2), turned to 270 degrees
- moved C23 5.08 mm to (68.6, 7.62)
- moved 10K_POT2 3.81 mm to (71.1, 15.2)
- moved 1M2 2.54 mm to (15.2, 12.7)
- moved LOW_BIT_NOISE 2.54 mm to (63.5, 57.1)
- moved FTDI 1.27 mm to (62.2, 52.1)
- moved JP2 1.27 mm to (31.8, 15.2)
- moved C6 1.27 mm to (74.9, 26.7)
- moved C7 1.27 mm to (71.1, 26.7)
- moved OK1 1.27 mm to (24.1, 16.5)
- moved R13 1.27 mm to (71.1, 21.6)
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Routing:
- net N$53: track 0.00 -> 100.6 mm
- net N$52: track 0.00 -> 38.9 mm
- net BD_TRIGGER: track 0.00 -> 31.6 mm, vias 0 -> 1
- net N$34: track 79.9 -> 109.7 mm
- net N$28: track 7.40 -> 29.6 mm
- net N$25: track 40.2 -> 60.8 mm
- net BD_OUT: track 155.6 -> 174.2 mm
- net N$51: track 6.66 -> 24.6 mm
- net GND: track 444.8 -> 431.9 mm, vias 1 -> 0
- net N$49: track 7.40 -> 19.4 mm
- net BD_OUT1: track 44.5 -> 51.4 mm
- net RESET: track 22.6 -> 28.2 mm
- net N$13: track 18.6 -> 22.7 mm
- net RX: track 3.81 -> 6.35 mm
- net N$60: track 8.15 -> 10.7 mm
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Other:
- board size 178.7 x 113 mm -> 107.6 x 78.7 mm

Commit message: long overdue commit
Parts:
- moved 10K_POT8 37.2 mm to (57.1, 6.35)
- moved LIMIT_SWITCH 37.2 mm to (50.8, 6.35), turned to 90 degrees
- moved R49 22.9 mm to (57.1, 8.89)
- moved Q3 20.7 mm to (102.9, 30.5), turned to 90 degrees
- moved R50 20.4 mm to (80.0, 11.4), turned to 180 degrees
- moved R6 17.1 mm to (19.1, 64.8)
- moved R26 13.0 mm to (80.0, 69.8)
- moved 10K_POT6 12.0 mm to (69.8, 68.6)
- moved C12 11.4 mm to (90.2, 69.8)
- moved D8 10.2 mm to (102.9, 19.1)
- moved 1M2 5.24 mm to (16.5, 17.8)
- moved 10K_POT 5.24 mm to (14.0, 54.6)
- moved LIM_SWITCH1 5.24 mm to (14.0, 61.0)
- moved R7 2.84 mm to (14.0, 45.7)
- moved D2 1.27 mm to (26.7, 8.89)
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Routing:
- net N$1: track 11.4 -> 48.6 mm
- net N$52: track 38.9 -> 8.67 mm
- net GND: track 431.9 -> 408.9 mm
- net N$51: track 24.6 -> 37.0 mm, vias 0 -> 1
- net N$59: track 13.8 -> 3.07 mm
- net BD_OUT: track 174.2 -> 163.5 mm
- net N$36: track 27.7 -> 38.2 mm
- net N$40: track 16.6 -> 25.5 mm
- net N$39: track 15.3 -> 6.88 mm
- net N$53: track 100.6 -> 108.8 mm
- net N$9: track 6.66 -> 13.5 mm
- net N$33: track 29.6 -> 23.5 mm
- net N$6: track 41.5 -> 35.4 mm
- net N$23: track 13.8 -> 8.45 mm
- net N$27: track 4.86 -> 9.42 mm
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Other:
- board size 107.6 x 78.7 mm -> 94.9 x 69.8 mm
